File: hardware/charger.kicad_sch (KiCad schematic)
At the start: 38 parts, among them J9 TYPE-C-31-M-12, Q1 SSM6J501NU, SW1 TS-1187A-B-A-B, U15 IP5328P

Commit message: update pcb
Parts:
- R124: footprint Resistor_SMD:R_0805_2012Metric -> Resistor_SMD:R_0603_1608Metric; chipdip 9000079478 -> (none); lcsc C17710 -> C23179
Changed lines of the file:
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@@
       (effects (font (size 1.27 1.27)) (justify right))
     )
-    (property "Footprint" "Resistor_SMD:R_0805_2012Metric" (id 2) (at 220.98 59.69 0)
+    (property "Footprint" "Resistor_SMD:R_0603_1608Metric" (id 2) (at 220.98 59.69 0)
       (effects (font (size 1.27 1.27)) hide)
     )
@@
       (effects (font (size 1.27 1.27)) hide)
     )
-    (property "chipdip" "9000079478" (id 4) (at 220.98 59.69 0)
+    (property "chipdip" "" (id 4) (at 220.98 59.69 0)
       (effects (font (size 1.27 1.27)) hide)
     )
@@
       (effects (font (size 1.27 1.27)) hide)
     )
-    (property "lcsc" "C17710" (id 6) (at 220.98 59.69 0)
+    (property "lcsc" "C23179" (id 6) (at 220.98 59.69 0)
       (effects (font (size 1.27 1.27)) hide)
     )

Commit message: update cap and dru
Parts:
- removed BT1, BT2, BT3, BT4: BH-18650-B1BA002, MAS_Package_nostd:BatteryHolder_BH-18650-B1BA002, symbol Device:Battery_Cell
- removed C180, C187, C188: 10u, Capacitor_SMD:C_0805_2012Metric, symbol Device:C_Small
- removed C181, C182: 2.2u, Capacitor_SMD:C_0805_2012Metric, symbol Device:C_Small
- removed F1, F2, F3, F4: 0466001.NRHF, MAS_Package_std:Fuse_1812_4532Metric, symbol Device:Fuse_Small
- added C52 (x4): 10u, Capacitor_SMD:C_0603_1608Metric, symbol Device:C_Small
- added C52: 4.7u, Capacitor_SMD:C_0603_1608Metric, symbol Device:C_Small
- C183, C184, C185: footprint Capacitor_SMD:C_0603_1608Metric -> Capacitor_SMD:C_0402_1005Metric; lcsc C14663 -> C307331
- JP1: value J_Boot -> JP; footprint Jumper:SolderJumper-2_P1.3mm_Open_Pad1.0x1.5mm -> MAS_Package_nostd:SolderJumper_Open_Pad0.5x0.8mm
- R115: footprint Resistor_SMD:R_0603_1608Metric -> Resistor_SMD:R_0402_1005Metric; lcsc C25804 -> C25744
- R116: footprint Resistor_SMD:R_0603_1608Metric -> Resistor_SMD:R_0402_1005Metric; lcsc C21190 -> C11702
- R118: footprint Resistor_SMD:R_0603_1608Metric -> Resistor_SMD:R_0402_1005Metric; lcsc C23254 -> C137932
- R119: footprint Resistor_SMD:R_0603_1608Metric -> Resistor_SMD:R_0402_1005Metric; lcsc C25803 -> C25741
- R121: footprint Resistor_SMD:R_0603_1608Metric -> Resistor_SMD:R_0402_1005Metric
- R122, R123: footprint Resistor_SMD:R_0603_1608Metric -> Resistor_SMD:R_0402_1005Metric; lcsc C23162 -> C25900
- R124: footprint Resistor_SMD:R_0603_1608Metric -> Resistor_SMD:R_0402_1005Metric; lcsc C23179 -> C25117
Connections:
- net +BATT: now also C52.1, C52.1, C52.2
- net -BATT: now also C52.1, C52.1, C52.2, C52.2, C52.2
- net VBUS: now also C52.1
- net VREG: now also C52.2
