File: hardware/main.kicad_pcb (KiCad board)
At the start: 2 copper layers, 88 x 111 mm, 502 parts, among them J1 DS1128-09-S8B8X, J2 DS1128-09-S8B8X, J3 DS1128-09-S8B8X, J4 SMA-KWE901, J5 SMA-KWE901, J6 IDC-08M, J7 IDC-08M, J8 USB_C_Receptacle, J9 TYPE-C-31-M-12, Q1 SSM6J501NU, Q2 SSM6J501NU, Q3 FDV301N, Q4 BC817, SW1 TS-1187A-B-A-B, SW2 TS-1187A-B-A-B, SW3 TS-1187A-B-A-B, SW4 TS-1187A-B-A-B, U1 SN74LVC1G175, U10 W25Q256FVEIG, U11 MT7603E, U12 TPD2EUSB30, U13 TPD2EUSB30, U14 TPD2EUSB30, U15 IP5328P, U16 N096-2864KSWEG01-H30, U2 MT7621A, U3 TPS63020, U4 TPS63020, U5 MT3420B, U6 MT3420B, U7 MT3420B, U8 MT3420B, U9 NT5CB64M16FP-DH (!), X1 HSO321S-50MHZ-3.3V, Y1 X322540MPB4SI

Commit message: update pcb
Parts:
- removed C111, C112, C113, C114: ~, Capacitor_SMD:C_0603_1608Metric
- removed C145: 100n, Capacitor_SMD:C_0603_1608Metric
- removed L10, L9: ~, Inductor_SMD:L_0603_1608Metric
- removed R68, R70: ~, Resistor_SMD:R_0603_1608Metric
- removed R69, R71: 0R, Resistor_SMD:R_0603_1608Metric
- C133, C134, C135, C136, C139, C195, C198, C199, C200, C201: footprint Capacitor_SMD:C_0805_2012Metric -> Capacitor_SMD:C_0603_1608Metric
- F1, F2, F3, F4, FID4, FID5, FID6: moved to B.Cu
- moved Y1 254.1 mm to (54.6, -61.0)
- moved C174 242.3 mm to (54.6, -64.1), turned to 180 degrees
- moved C175 235.8 mm to (54.6, -57.8)
- moved R100 231.7 mm to (54.6, -66.7)
- moved C69 209.7 mm to (26.0, -85.7)
- moved C62 208.2 mm to (22.2, -85.1)
- moved C60 208.1 mm to (22.2, -87.0)
- moved C57 206.6 mm to (26.0, -87.6)
- moved C74 205.7 mm to (22.2, -79.4)
- moved C65 204.9 mm to (22.2, -81.3)
- moved C76 203.3 mm to (50.2, -84.1), turned to 90 degrees
- moved TP1 203.0 mm to (14.0, -77.5)
- moved TP3 202.3 mm to (14.0, -73.7)
- moved C70 202.0 mm to (22.2, -83.2)
- moved C67 201.8 mm to (26.0, -81.9)
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Connections:
- C115 pad 1: Net-(C113-Pad1) -> Net-(C115-Pad1)
- C116 pad 1: Net-(C114-Pad1) -> Net-(C116-Pad1)
- J4 pad 1: Net-(C111-Pad1) -> Net-(C115-Pad1)
- J5 pad 1: Net-(C112-Pad1) -> Net-(C116-Pad1)
- L11 pad 1: Net-(C113-Pad1) -> Net-(C115-Pad1)
- L12 pad 1: Net-(C114-Pad1) -> Net-(C116-Pad1)
- TP25 pad 1: /Interface/PCIE_CK1_P -> /Interface/PCIE_CK0_P
- TP26 pad 1: /Interface/PCIE_CK1_N -> /Interface/PCIE_CK0_N
- TP27 pad 1: /Interface/PCIE_TX1_P -> /Interface/PCIE_TX0_P
- TP28 pad 1: /Interface/PCIE_TX1_N -> /Interface/PCIE_TX0_N
- TP29 pad 1: /Interface/PCIE_RX1_P -> /Interface/PCIE_RX0_P
- TP30 pad 1: /Interface/PCIE_RX1_N -> /Interface/PCIE_RX0_N

Commit message: update pcb
Parts:
- R124, R126, R5: footprint Resistor_SMD:R_0805_2012Metric -> Resistor_SMD:R_0603_1608Metric
- moved J8 289.7 mm to (57.8, -132.7), turned to 180 degrees
- moved R101 280.1 mm to (60.3, -126.4), turned to 0 degrees
- moved U14 276.7 mm to (60.3, -124.5), turned to 180 degrees
- moved R102 276.0 mm to (55.2, -126.4), turned to 180 degrees
- moved U12 274.5 mm to (57.8, -124.5), turned to 180 degrees
- moved U13 272.5 mm to (55.2, -124.5), turned to 180 degrees
- moved C160 271.2 mm to (61.0, -121.1), turned to 90 degrees
- moved FID1 270.4 mm to (101.2, -133.9)
- moved FID2 270.4 mm to (97.0, -138.5)
- moved FID3 270.4 mm to (96.7, -133.9)
- moved FID4 270.4 mm to (112.8, -138.5)
- moved FID5 270.4 mm to (117.4, -133.4)
- moved FID6 270.4 mm to (117.4, -138.5)
- moved H3 270.4 mm to (90.8, -137.2)
- moved H4 270.4 mm to (83.7, -137.2)
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Connections:
- SW2 pad 1: Net-(C9-Pad1) -> -BATT
- SW2 pad 2: -BATT -> Net-(C9-Pad1)

Commit message: trace ram
Parts:
- C57, C58, C60, C61, C62, C63, C64, C65, C67, C68, C69, C70, C72, C74: moved to B.Cu
- moved C73 133.1 mm to (20.8, -53.8), turned to 180 degrees
- moved R35 132.9 mm to (22.1, -65.3), turned to 0 degrees
- moved R20 132.1 mm to (20.8, -52.3), turned to 0 degrees
- moved R15 131.3 mm to (20.8, -50.8), turned to 180 degrees
- moved R14 131.2 mm to (22.1, -68.3), turned to 0 degrees
- moved R3 131.0 mm to (20.8, -55.4), turned to 0 degrees
- moved C66 130.1 mm to (22.1, -66.8), turned to 180 degrees
- moved R13 129.3 mm to (22.1, -69.8), turned to 180 degrees
- moved C64 123.5 mm to (24.8, -70.5), turned to 90 degrees
- moved C63 123.2 mm to (24.8, -67.3), turned to 90 degrees
- moved C72 121.6 mm to (24.8, -61.0), turned to -90 degrees
- moved C74 121.0 mm to (24.8, -64.1), turned to 90 degrees
- moved C65 120.8 mm to (27.9, -61.0), turned to 90 degrees
- moved C60 120.7 mm to (29.6, -64.1), turned to -90 degrees
- moved C67 120.4 mm to (27.3, -70.5), turned to 90 degrees
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Routing:
- net +1V5: track 0.00 -> 82.4 mm, vias 0 -> 18
- net /Memory/RA4: track 0.00 -> 47.2 mm
- net /Memory/RA6: track 0.00 -> 42.0 mm
- net /Memory/RA8: track 0.00 -> 40.5 mm
- net /Memory/RA11: track 0.00 -> 38.2 mm
- net /Memory/RA12: track 0.00 -> 37.7 mm
- net /Memory/RCKE: track 0.00 -> 37.2 mm
- net /Memory/RBA1: track 0.00 -> 36.6 mm
- net /Memory/RA14: track 0.00 -> 36.4 mm
- net /Memory/RA1: track 0.00 -> 35.8 mm
- net /Memory/RA5: track 0.00 -> 28.5 mm
- net /Memory/RBA0: track 0.00 -> 27.8 mm
- net /Memory/RA7: track 0.00 -> 27.2 mm, vias 0 -> 2
- net /Memory/RA3: track 0.00 -> 27.0 mm
- net /Memory/~{RCLK}: track 0.00 -> 26.3 mm, vias 0 -> 3
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- added copper zone on B.Cu, net -BATT
- added copper zone on F.Cu, net -BATT
Other:
- copper layers 2 -> 4

Commit message: fix pcb
Parts:
- added C174: 18p, Capacitor_SMD:C_0603_1608Metric, F.Cu at (150.1, -51.4)
- added C175: 18p, Capacitor_SMD:C_0603_1608Metric, F.Cu at (150.1, -45.0)
- added C57: 100n, Capacitor_SMD:C_0603_1608Metric, B.Cu at (143.7, -69.8)
- added C58: 100n, Capacitor_SMD:C_0603_1608Metric, B.Cu at (139.1, -60.3)
- added C59: 100n, Capacitor_SMD:C_0603_1608Metric, B.Cu at (146.1, -62.9)
- added C60: 100n, Capacitor_SMD:C_0603_1608Metric, B.Cu at (139.1, -63.4)
- added C61: 100n, Capacitor_SMD:C_0603_1608Metric, B.Cu at (143.7, -60.3)
- added C62: 100n, Capacitor_SMD:C_0603_1608Metric, B.Cu at (141.2, -69.8)
- added C63: 100n, Capacitor_SMD:C_0603_1608Metric, B.Cu at (134.2, -66.6)
- added C64: 100n, Capacitor_SMD:C_0603_1608Metric, B.Cu at (134.2, -69.8)
- added C65: 100n, Capacitor_SMD:C_0603_1608Metric, B.Cu at (137.4, -60.3)
- added C66: 100n, Capacitor_SMD:C_0603_1608Metric, F.Cu at (131.5, -66.1)
- added C67: 100n, Capacitor_SMD:C_0603_1608Metric, B.Cu at (136.8, -69.8)
- added C68: 100n, Capacitor_SMD:C_0603_1608Metric, B.Cu at (141.2, -66.6)
- added C69: 100n, Capacitor_SMD:C_0603_1608Metric, B.Cu at (143.7, -66.6)
- added C70: 100n, Capacitor_SMD:C_0603_1608Metric, B.Cu at (143.7, -63.4)
- added C71: 100n, Capacitor_SMD:C_0603_1608Metric, B.Cu at (146.1, -59.9)
- added C72: 100n, Capacitor_SMD:C_0603_1608Metric, B.Cu at (134.2, -60.3)
- added C73: 100n, Capacitor_SMD:C_0603_1608Metric, F.Cu at (130.3, -53.1)
- added C74: 100n, Capacitor_SMD:C_0603_1608Metric, B.Cu at (134.2, -63.4)
- added C75: 4.7u, Capacitor_SMD:C_0805_2012Metric, F.Cu at (132.1, -71.7)
- added C76: 4.7u, Capacitor_SMD:C_0805_2012Metric, F.Cu at (130.0, -71.7)
- added R10: 1k, Resistor_SMD:R_0603_1608Metric, B.Cu at (146.1, -61.4)
- added R100: 24k, Resistor_SMD:R_0603_1608Metric, F.Cu at (152.6, -53.6)
- added R11: 1k, Resistor_SMD:R_0603_1608Metric, B.Cu at (146.1, -64.4)
- added R13: 1k, Resistor_SMD:R_0603_1608Metric, F.Cu at (131.5, -69.1)
- added R14: 1k, Resistor_SMD:R_0603_1608Metric, F.Cu at (131.5, -67.6)
- added R15: 1k, Resistor_SMD:R_0603_1608Metric, F.Cu at (130.3, -50.1)
- added R20: 1k, Resistor_SMD:R_0603_1608Metric, F.Cu at (130.3, -51.6)
- added R3: 0R, Resistor_SMD:R_0603_1608Metric, F.Cu at (130.3, -54.7)
- added R34: 100R, Resistor_SMD:R_0603_1608Metric, F.Cu at (131.5, -63.0)
- added R35: 240R, Resistor_SMD:R_0603_1608Metric, F.Cu at (131.5, -64.6)
- added U2: MT7621A, MAS_Package_std:TFBGA-387_11.7x13.6mm_P0.65mm, F.Cu at (138.8, -47.8)
- added U9: NT5CB64M16FP-DH (!), Package_BGA:BGA-96_9.0x13.0mm_Layout2x3x16_P0.8mm, F.Cu at (138.8, -65.5)
- added Y1: X322540MPB4SI, MAS_Package_std:Oscillator_SMD_SMD3225-4P, F.Cu at (150.1, -48.2)
- C59, C71, R10, R11: moved to B.Cu
- moved C59 0.12 mm to (36.6, -63.6), turned to 180 degrees
- moved C71 0.12 mm to (36.6, -60.6), turned to 0 degrees
- moved R10 0.12 mm to (36.6, -62.1), turned to 180 degrees
- moved R11 0.12 mm to (36.6, -65.1), turned to 0 degrees
Routing:
- net /Memory/RCLK: track 24.8 -> 105.9 mm, vias 3 -> 6
- net +1V5: track 82.4 -> 162.0 mm, vias 18 -> 34
- net /Memory/~{RCLK}: track 26.3 -> 105.7 mm, vias 3 -> 6
- net /Memory/RA3: track 27.0 -> 96.6 mm
- net /Memory/~{RCS}: track 25.1 -> 89.7 mm
- net /Memory/~{RWE}: track 26.2 -> 89.9 mm
- net /Memory/RBA0: track 27.8 -> 90.2 mm
- net /Memory/RA5: track 28.5 -> 89.6 mm
- net /Memory/RA4: track 47.2 -> 103.5 mm
- net /Memory/~{RRAS}: track 24.6 -> 80.9 mm
- net /Memory/RA1: track 35.8 -> 89.9 mm
- net /Memory/RA14: track 36.4 -> 89.9 mm
- net /Memory/RBA1: track 36.6 -> 90.0 mm
- net /Memory/RCKE: track 37.2 -> 90.1 mm
- net /Memory/RA12: track 37.7 -> 89.7 mm
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
Commit message: update cap and dru
Parts:
- removed BT1, BT2, BT3, BT4: BH-18650-B1BA002, MAS_Package_nostd:BatteryHolder_BH-18650-B1BA002
- removed C115, C116: 9p, Capacitor_SMD:C_0603_1608Metric
- removed C117, C118, C119, C120: 1.2p, Capacitor_SMD:C_0603_1608Metric
- removed C121, C122, C123, C124: 10p, Capacitor_SMD:C_0603_1608Metric
- removed C125, C126, C127, C128: 0.5p, Capacitor_SMD:C_0603_1608Metric
- removed C129, C130, C131, C132: 3p, Capacitor_SMD:C_0603_1608Metric
- removed C133, C134, C135, C136, C139: 1u, Capacitor_SMD:C_0603_1608Metric
- removed C137, C140, C143, C144, C146, C147, C148, C149, C150, C153, C154, C155, C156: 100n, Capacitor_SMD:C_0603_1608Metric
- removed C138: 22u, Capacitor_SMD:C_0805_2012Metric
- removed C141, C152: 10u, Capacitor_SMD:C_0805_2012Metric
- removed C142: 4.7u, Capacitor_SMD:C_0805_2012Metric
- removed C151, C157: 2.2u, Capacitor_SMD:C_0805_2012Metric
- removed the C174 at (150.1, -51.4)
- removed the C175 at (150.1, -45.0)
- removed the C57 at (143.7, -69.8)
- removed the C58 at (139.1, -60.3)
- removed the C59 at (146.1, -62.9)
- removed the C60 at (139.1, -63.4)
- removed the C61 at (143.7, -60.3)
- removed the C62 at (141.2, -69.8)
- removed the C63 at (134.2, -66.6)
- removed the C64 at (134.2, -69.8)
- removed the C65 at (137.4, -60.3)
- removed the C66 at (131.5, -66.1)
- removed the C67 at (136.8, -69.8)
- removed the C68 at (141.2, -66.6)
- removed the C69 at (143.7, -66.6)
- removed the C70 at (143.7, -63.4)
- removed the C71 at (146.1, -59.9)
- removed the C72 at (134.2, -60.3)
- removed the C73 at (130.3, -53.1)
- removed the C74 at (134.2, -63.4)
- removed the C75 at (132.1, -71.7)
- removed the C76 at (130.0, -71.7)
- removed F3, F4: 0466001.NRHF, MAS_Package_std:Fuse_1812_4532Metric
- removed J5: SMA-KWE901, MAS_Package_std:SMA_Amphenol_901-143_Horizontal
- removed L11, L12: SDCL1608C1N2STDF, Inductor_SMD:L_0603_1608Metric
- removed L13, L14, L15, L16: HK16082N7S-T, Inductor_SMD:L_0603_1608Metric
- removed L17, L18, L19, L20: VHF160808H1N8ST, Inductor_SMD:L_0603_1608Metric
- removed L21, L22, L23, L24: SDCL1608C3N0STDF, Inductor_SMD:L_0603_1608Metric
- removed L25: SLO0530H2R2MTT, MAS_Package_std:Power_inductor_SMD_0530
- removed the R10 at (146.1, -61.4)
- removed the R100 at (152.6, -53.6)
- removed the R11 at (146.1, -64.4)
- removed the R13 at (131.5, -69.1)
- removed the R14 at (131.5, -67.6)
- removed the R15 at (130.3, -50.1)
- removed the R20 at (130.3, -51.6)
- removed the R3 at (130.3, -54.7)
- removed the R34 at (131.5, -63.0)
- removed the R35 at (131.5, -64.6)
- removed R72, R81, R86: 0R, Resistor_SMD:R_0603_1608Metric
- removed R73, R76, R78, R79, R82, R83, R84, R85, R88: ~, Resistor_SMD:R_0603_1608Metric
- removed R74, R75, R77, R80, R87: 4.7k, Resistor_SMD:R_0603_1608Metric
- removed R89: 5.1k, Resistor_SMD:R_0603_1608Metric
- removed TP15, TP16, TP17, TP18, TP25, TP26, TP27, TP28, TP29, TP30: TestPoint, TestPoint:TestPoint_Pad_D1.0mm
- removed U11: MT7603E, MAS_Package_std:QFN-56-1EP_7x7mm_P0.4mm_EP4.6x4.6mm
- removed the U2 at (138.8, -47.8)
- removed the U9 at (138.8, -65.5)
- removed X1: HSO321S-50MHZ-3.3V, MAS_Package_std:Oscillator_SMD_SMD3225-4P
- removed the Y1 at (150.1, -48.2)
- C1, C103, C17, C180, C187, C188, C202, C203, C23, C36, C37, C4, C45, C46, C47, C48, C5, C55, C56, C6, C7, C75, C76, C81, C82, C85: footprint Capacitor_SMD:C_0805_2012Metric -> Capacitor_SMD:C_0603_1608Metric
- C10, C100, C101, C102, C104, C106, C109, C11, C110, C12, C13, C159, C16, C160, C161, C162, C163, C164, C165, C166, C167, C168, C169, C170, C171, C172, C173, C174, C175, C176, C177, C178, C179, C18, C183, C184, C185, C19, C193, C194, C196, C197, C2, C20, C21, C22, C24, C25, C26, C27, C28, C29, C3, C38, C39, C40, C41, C42, C43, C44, C49, C50, C51, C52, C53, C54, C57, C58, C59, C60, C61, C62, C63, C64, C65, C66, C67, C68, C69, C70, C71, C72, C73, C74, C77, C78, C79, C8, C80, C83, C84, C86, C87, C88, C89, C9, C90, C91, C92, C93, C94, C95, C96, C97, C98, C99: footprint Capacitor_SMD:C_0603_1608Metric -> Capacitor_SMD:C_0402_1005Metric
- C14, C15, C182, C30, C31, C32, C33: value 2.2u -> 4.7u; footprint Capacitor_SMD:C_0805_2012Metric -> Capacitor_SMD:C_0603_1608Metric
- C158: value 10u -> 4.7u; footprint Capacitor_SMD:C_0805_2012Metric -> Capacitor_SMD:C_0603_1608Metric
- C181: value 2.2u -> 10u; footprint Capacitor_SMD:C_0805_2012Metric -> Capacitor_SMD:C_0603_1608Metric
- C195, C198, C199, C200, C201: value 1u -> 4.7u
- F1, F2: value 0466001.NRHF -> 12T.30000063AG12S1B02; footprint MAS_Package_std:Fuse_1812_4532Metric -> Fuse:Fuse_1206_3216Metric
- J4: value SMA-KWE901 -> 98424-G52-04ALF; footprint MAS_Package_std:SMA_Amphenol_901-143_Horizontal -> MAS_Package_std:PinSocket_2x02_P2.00mm_Vertical_SMD; moved to F.Cu
- JP1, JP2, JP3, JP4, JP5, JP6, JP7: value J_Boot -> JP; footprint Jumper:SolderJumper-2_P1.3mm_Open_Pad1.0x1.5mm -> MAS_Package_nostd:SolderJumper_Open_Pad0.5x0.8mm
- R1, R10, R100, R101, R102, R103, R104, R105, R106, R107, R108, R109, R11, R110, R111, R112, R113, R114, R115, R116, R118, R119, R12, R121, R122, R123, R124, R125, R126, R127, R128, R129, R13, R130, R131, R132, R133, R134, R135, R136, R137, R138, R139, R14, R140, R141, R142, R143, R144, R145, R146, R147, R148, R149, R15, R150, R151, R152, R153, R154, R155, R156, R157, R158, R159, R16, R160, R161, R162, R163, R164, R165, R166, R167, R168, R169, R17, R170, R171, R172, R18, R19, R2, R20, R21, R22, R23, R24, R25, R26, R27, R28, R29, R3, R30, R31, R32, R33, R34, R35, R36, R37, R38, R39, R4, R40, R41, R42, R43, R44, R45, R46, R47, R48, R49, R5, R50, R51, R52, R53, R54, R55, R56, R57, R58, R59, R6, R60, R61, R62, R63, R64, R65, R66, R67, R7, R8, R9, R90, R91, R92, R93, R94, R95, R96, R97, R98, R99: footprint Resistor_SMD:R_0603_1608Metric -> Resistor_SMD:R_0402_1005Metric
- TP1, TP10, TP11, TP12, TP13, TP14, TP19, TP2, TP20, TP21, TP22, TP23, TP24, TP3, TP31, TP32, TP33, TP34, TP4, TP5, TP6, TP7, TP8, TP9: value TestPoint -> TP
- moved C77 206.3 mm to (-52.5, -1.42)
- moved R41 206.3 mm to (-47.4, -1.42)
- moved TP4 206.3 mm to (-57.5, -14.1)
- moved TP5 206.3 mm to (-57.5, -12.2)
- moved TP6 206.3 mm to (-57.5, -10.3)
- moved TP7 206.3 mm to (-57.5, -8.41)
- moved TP8 206.3 mm to (-57.5, -6.50)
- moved R2 206.3 mm to (-39.1, -10.9)
- moved R40 206.3 mm to (-48.0, -10.9)
- moved R42 206.3 mm to (-49.9, -10.9)
- moved R43 206.3 mm to (-46.1, -10.9)
- moved R8 206.3 mm to (-40.8, -4.60)
- moved R9 206.3 mm to (-40.8, -7.77)
- moved TP1 206.3 mm to (-57.5, -19.8)
- moved TP2 206.3 mm to (-57.5, -17.9)
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Connections:
- net Net-(J1-Pad1) renamed /Ethernet/P4A_P
- net Net-(J1-Pad2) renamed /Ethernet/P4A_N
- net Net-(J1-Pad3) renamed /Ethernet/P4B_P
- net Net-(J1-Pad4) renamed /Ethernet/P4C_P
- net Net-(J1-Pad5) renamed /Ethernet/P4C_N
- net Net-(J1-Pad6) renamed /Ethernet/P4B_N
- net Net-(J1-Pad7) renamed /Ethernet/P4D_P
- net Net-(J1-Pad8) renamed /Ethernet/P4D_N
- net Net-(J2-Pad1) renamed /Ethernet/P3A_P
- net Net-(J2-Pad2) renamed /Ethernet/P3A_N
- net Net-(J2-Pad3) renamed /Ethernet/P3B_P
- net Net-(J2-Pad4) renamed /Ethernet/P3C_P
- net Net-(J2-Pad5) renamed /Ethernet/P3C_N
- net Net-(J2-Pad6) renamed /Ethernet/P3B_N
- net Net-(J2-Pad7) renamed /Ethernet/P3D_P
- net Net-(J2-Pad8) renamed /Ethernet/P3D_N
- net Net-(J3-Pad1) renamed /Ethernet/P2A_P
- net Net-(J3-Pad2) renamed /Ethernet/P2A_N
- net Net-(J3-Pad3) renamed /Ethernet/P2B_P
- net Net-(J3-Pad4) renamed /Ethernet/P2C_P
- net Net-(J3-Pad5) renamed /Ethernet/P2C_N
- net Net-(J3-Pad6) renamed /Ethernet/P2B_N
- net Net-(J3-Pad7) renamed /Ethernet/P2D_P
- net Net-(J3-Pad8) renamed /Ethernet/P2D_N
- F1 pad 1: Net-(BT1-Pad1) -> Net-(J4-Pin_3)
- F2 pad 1: Net-(BT2-Pad1) -> Net-(J4-Pin_4)
- J1 pad 11: /Ethernet/Y0- -> /Ethernet/Y2-
- J1 pad 9: /Ethernet/G0- -> /Ethernet/G2-
- J2 pad 11: /Ethernet/Y1- -> /Ethernet/Y3-
- J2 pad 9: /Ethernet/G1- -> /Ethernet/G3-
- J3 pad 11: /Ethernet/Y1- -> /Ethernet/Y4-
- J3 pad 9: /Ethernet/G1- -> /Ethernet/G4-
- J4 pad 1: Net-(C115-Pad1) -> -BATT
- TR1 pad 1: /Ethernet/ESW_TXVN_D_P0 -> /Ethernet/ESW_TXVN_D_P2
- TR1 pad 11: /Ethernet/ESW_TXVN_A_P0 -> /Ethernet/ESW_TXVN_A_P2
- TR1 pad 12: /Ethernet/ESW_TXVP_A_P0 -> /Ethernet/ESW_TXVP_A_P2
- TR1 pad 2: /Ethernet/ESW_TXVP_D_P0 -> /Ethernet/ESW_TXVP_D_P2
- TR1 pad 5: /Ethernet/ESW_TXVN_C_P0 -> /Ethernet/ESW_TXVN_C_P2
- TR1 pad 6: /Ethernet/ESW_TXVP_C_P0 -> /Ethernet/ESW_TXVP_C_P2
- TR1 pad 7: /Ethernet/ESW_TXVN_B_P0 -> /Ethernet/ESW_TXVN_B_P2
- TR1 pad 8: /Ethernet/ESW_TXVP_B_P0 -> /Ethernet/ESW_TXVP_B_P2
- TR2 pad 1: /Ethernet/ESW_TXVN_D_P1 -> /Ethernet/ESW_TXVN_D_P3
- TR2 pad 11: /Ethernet/ESW_TXVN_A_P1 -> /Ethernet/ESW_TXVN_A_P3
- TR2 pad 12: /Ethernet/ESW_TXVP_A_P1 -> /Ethernet/ESW_TXVP_A_P3
- TR2 pad 2: /Ethernet/ESW_TXVP_D_P1 -> /Ethernet/ESW_TXVP_D_P3
- TR2 pad 5: /Ethernet/ESW_TXVN_C_P1 -> /Ethernet/ESW_TXVN_C_P3
- TR2 pad 6: /Ethernet/ESW_TXVP_C_P1 -> /Ethernet/ESW_TXVP_C_P3
- TR2 pad 7: /Ethernet/ESW_TXVN_B_P1 -> /Ethernet/ESW_TXVN_B_P3
- TR2 pad 8: /Ethernet/ESW_TXVP_B_P1 -> /Ethernet/ESW_TXVP_B_P3
- TR3 pad 1: /Ethernet/ESW_TXVN_D_P2 -> /Ethernet/ESW_TXVN_D_P4
- TR3 pad 11: /Ethernet/ESW_TXVN_A_P2 -> /Ethernet/ESW_TXVN_A_P4
- TR3 pad 12: /Ethernet/ESW_TXVP_A_P2 -> /Ethernet/ESW_TXVP_A_P4
- TR3 pad 2: /Ethernet/ESW_TXVP_D_P2 -> /Ethernet/ESW_TXVP_D_P4
- TR3 pad 5: /Ethernet/ESW_TXVN_C_P2 -> /Ethernet/ESW_TXVN_C_P4
- TR3 pad 6: /Ethernet/ESW_TXVP_C_P2 -> /Ethernet/ESW_TXVP_C_P4
- TR3 pad 7: /Ethernet/ESW_TXVN_B_P2 -> /Ethernet/ESW_TXVN_B_P4
- TR3 pad 8: /Ethernet/ESW_TXVP_B_P2 -> /Ethernet/ESW_TXVP_B_P4
- U2 pad AA10: unconnected-(U2-PadAA10) -> /Ethernet/ESW_TXVN_C_P3
- U2 pad AA11: unconnected-(U2-PadAA11) -> /Ethernet/ESW_TXVP_A_P4
- U2 pad AA13: unconnected-(U2-PadAA13) -> /Ethernet/ESW_TXVP_C_P4
- U2 pad AA15: /Ethernet/P3_LED_0 -> /Ethernet/G3-
- U2 pad AA17: /Ethernet/G0- -> /Ethernet/P0_LED_0
- U2 pad R2: /Ethernet/ESW_TXVP_B_P0 -> unconnected-(U2D-ESW_TXVP_B_P0-PadR2)
- U2 pad R3: /Ethernet/ESW_TXVN_B_P0 -> unconnected-(U2D-ESW_TXVN_B_P0-PadR3)
- U2 pad R5: /Ethernet/ESW_TXVN_A_P0 -> unconnected-(U2D-ESW_TXVN_A_P0-PadR5)
- U2 pad T2: /Ethernet/ESW_TXVP_C_P0 -> unconnected-(U2D-ESW_TXVP_C_P0-PadT2)
- U2 pad T3: /Ethernet/ESW_TXVN_C_P0 -> unconnected-(U2D-ESW_TXVN_C_P0-PadT3)
- U2 pad T4: /Ethernet/ESW_TXVP_A_P1 -> unconnected-(U2D-ESW_TXVP_A_P1-PadT4)
- U2 pad T5: /Ethernet/ESW_TXVP_A_P0 -> unconnected-(U2D-ESW_TXVP_A_P0-PadT5)
- U2 pad U1: /Ethernet/ESW_TXVP_D_P0 -> unconnected-(U2D-ESW_TXVP_D_P0-PadU1)
- U2 pad U2: /Ethernet/ESW_TXVN_D_P0 -> unconnected-(U2D-ESW_TXVN_D_P0-PadU2)
- U2 pad U4: /Ethernet/ESW_TXVN_A_P1 -> unconnected-(U2D-ESW_TXVN_A_P1-PadU4)
- U2 pad V10: unconnected-(U2-PadV10) -> /Ethernet/ESW_TXVP_D_P3
- U2 pad V2: /Ethernet/ESW_TXVP_B_P1 -> unconnected-(U2D-ESW_TXVP_B_P1-PadV2)
- U2 pad V3: /Ethernet/ESW_TXVN_B_P1 -> unconnected-(U2D-ESW_TXVN_B_P1-PadV3)
- U2 pad W1: /Ethernet/ESW_TXVP_C_P1 -> unconnected-(U2D-ESW_TXVP_C_P1-PadW1)
- U2 pad W10: unconnected-(U2-PadW10) -> /Ethernet/ESW_TXVN_D_P3
- U2 pad W12: unconnected-(U2-PadW12) -> /Ethernet/ESW_TXVN_B_P4
- U2 pad W14: unconnected-(U2-PadW14) -> /Ethernet/ESW_TXVP_D_P4
- U2 pad W2: /Ethernet/ESW_TXVN_C_P1 -> unconnected-(U2D-ESW_TXVN_C_P1-PadW2)
- U2 pad W8: unconnected-(U2-PadW8) -> /Ethernet/ESW_TXVP_A_P3
- U2 pad W9: unconnected-(U2-PadW9) -> /Ethernet/ESW_TXVP_B_P3
- U2 pad Y1: /Ethernet/ESW_TXVP_D_P1 -> unconnected-(U2D-ESW_TXVP_D_P1-PadY1)
- U2 pad Y10: unconnected-(U2-PadY10) -> /Ethernet/ESW_TXVP_C_P3
- U2 pad Y11: unconnected-(U2-PadY11) -> /Ethernet/ESW_TXVN_A_P4
- U2 pad Y12: unconnected-(U2-PadY12) -> /Ethernet/ESW_TXVP_B_P4
- U2 pad Y13: unconnected-(U2-PadY13) -> /Ethernet/ESW_TXVN_C_P4
- U2 pad Y14: unconnected-(U2-PadY14) -> /Ethernet/ESW_TXVN_D_P4
- U2 pad Y15: /Ethernet/P4_LED_0 -> /Ethernet/G4-
- U2 pad Y16: /Ethernet/G1- -> /Ethernet/P1_LED_0
- U2 pad Y2: /Ethernet/ESW_TXVN_D_P1 -> unconnected-(U2D-ESW_TXVN_D_P1-PadY2)
- U2 pad Y8: unconnected-(U2-PadY8) -> /Ethernet/ESW_TXVN_A_P3
- U2 pad Y9: unconnected-(U2-PadY9) -> /Ethernet/ESW_TXVN_B_P3
Routing:
- net +1V5: track 162.0 -> 0.00 mm, vias 34 -> 0
- net /Memory/RCLK: track 105.9 -> 0.00 mm, vias 6 -> 0
- net /Memory/~{RCLK}: track 105.7 -> 0.00 mm, vias 6 -> 0
- net /Memory/RA4: track 103.5 -> 0.00 mm
- net /Memory/RA3: track 96.6 -> 0.00 mm
- net /Memory/RA6: track 90.4 -> 0.00 mm
- net /Memory/RA8: track 90.2 -> 0.00 mm
- net /Memory/RBA0: track 90.2 -> 0.00 mm
- net /Memory/RCKE: track 90.1 -> 0.00 mm
- net /Memory/RA11: track 90.1 -> 0.00 mm
- net /Memory/RBA1: track 90.0 -> 0.00 mm
- net /Memory/~{RWE}: track 89.9 -> 0.00 mm
- net /Memory/RA1: track 89.9 -> 0.00 mm
- net /Memory/RA14: track 89.9 -> 0.00 mm
- net /Memory/RA12: track 89.7 -> 0.00 mm
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- removed copper zone on B.Cu, net -BATT
