File: hardware/main.kicad_pcb (KiCad board)
At the start: 4 copper layers, 57 x 93 mm, 414 parts, among them J1 DS1128-09-S8B8X, J10 AS0BC21-S30BM-7H, J2 DS1128-09-S8B8X, J3 DS1128-09-S8B8X, J4 98424-G52-04ALF, J5 miniPCI-E_52P_5.2, J6 IDC-08M, J7 IDC-08M, J8 USB_C_Receptacle, J9 TYPE-C-31-M-12, Q1 SSM6J501NU, Q2 SSM6J501NU, Q3 FDV301N, SW1 TS-1187A-B-A-B, SW2 TS-1187A-B-A-B, U1 SSD1306-OLED-0.91, U10 W25Q256FVEIG, U12 TPD2EUSB30, U13 TPD2EUSB30, U14 TPD2EUSB30, U15 IP5328P, U2 MT7621A, U3 TPS63020, U4 TPS63020, U5 MT3420B, U6 MT3420B, U7 MT3420B, U8 MT3420B, U9 NT5CB64M16FP-DH (!), Y1 X322540MPB4SI

Commit message: update sch
Parts:
- removed Q2: SSM6J501NU, MAS_Package_std:U-MOSVI
- removed RN1: 4D03WGJ0102T5E, Resistor_SMD:R_Array_Convex_4x0603
- added C133: 100n, Capacitor_SMD:C_0402_1005Metric, B.Cu at (72.1, -70.5)
- added C137: 33p, Capacitor_SMD:C_0402_1005Metric, B.Cu at (72.1, -68.6)
- added C138: 33p, Capacitor_SMD:C_0402_1005Metric, B.Cu at (72.1, -66.6)
- added C142: 33p, Capacitor_SMD:C_0402_1005Metric, B.Cu at (72.1, -64.6)
- added D5: MBR0540, Diode_SMD:D_SOD-123, B.Cu at (28.4, -85.5)
- added R126: 4.7k, Resistor_SMD:R_0402_1005Metric, F.Cu at (43.3, -82.2)
- added R127: 4.7k, Resistor_SMD:R_0402_1005Metric, F.Cu at (43.3, -80.2)
- added R162: 4.7k, Resistor_SMD:R_0402_1005Metric, F.Cu at (43.3, -78.2)
- added R163: 4.7k, Resistor_SMD:R_0402_1005Metric, F.Cu at (43.3, -76.2)
- added R88: 0R, Resistor_SMD:R_0402_1005Metric, B.Cu at (44.3, -65.2)
- added R89: 0R, Resistor_SMD:R_0402_1005Metric, B.Cu at (44.3, -63.2)
- added R98: 330k, Resistor_SMD:R_0402_1005Metric, B.Cu at (27.0, -88.1)
- added R99: 10k, Resistor_SMD:R_0402_1005Metric, B.Cu at (27.0, -90.1)
- added TP20: TP, MAS_Package_std:TestPoint_Pad_D1mm, B.Cu at (44.7, -61.1)
- added TP21: TP, MAS_Package_std:TestPoint_Pad_D1mm, B.Cu at (44.7, -59.0)
- added TP22: TP, MAS_Package_std:TestPoint_Pad_D1mm, B.Cu at (21.6, -37.6)
- added TP32: TP, MAS_Package_std:TestPoint_Pad_D1mm, B.Cu at (21.6, -35.4)
- added TP33: TP, MAS_Package_std:TestPoint_Pad_D1mm, B.Cu at (21.6, -33.3)
- added TP34: TP, MAS_Package_std:TestPoint_Pad_D1mm, B.Cu at (21.6, -31.2)
- C2: value 100n -> 10u; footprint Capacitor_SMD:C_0402_1005Metric -> Capacitor_SMD:C_0603_1608Metric
- C24, C28, C32, C5, R18, R19: moved to F.Cu
- J6: value IDC-08M -> 1042240820; footprint Connector_PinHeader_1.27mm:PinHeader_2x04_P1.27mm_Vertical -> MAS_Package_std:1042240820
- J7: value IDC-08M -> ~; footprint Connector_PinHeader_1.27mm:PinHeader_2x04_P1.27mm_Vertical -> Connector_PinHeader_1.27mm:PinHeader_2x05_P1.27mm_Vertical
- R1: value 1k -> 22R
- R4: value 10k -> 1k
- R5: value 470R -> 22R
- R7: value 1k -> 470R
- R80, R81, R82, R83, R84, R85: moved to B.Cu
- moved C7 53.4 mm to (17.4, -49.9)
- moved J6 28.0 mm to (64.1, -76.2)
- moved C32 12.3 mm to (43.0, -87.6), turned to 180 degrees
- moved R80 9.95 mm to (43.1, -31.6)
- moved R85 9.95 mm to (33.1, -31.6)
- moved R81 5.97 mm to (41.1, -31.6)
- moved R84 5.97 mm to (35.1, -31.6)
- moved C5 5.43 mm to (7.87, -74.0), turned to 180 degrees
- moved C33 4.78 mm to (6.86, -65.8), turned to 0 degrees
- moved R24 3.44 mm to (4.70, -66.8), turned to -90 degrees
- moved JP6 3.41 mm to (8.76, -63.6)
- moved C28 2.33 mm to (1.14, -66.2), turned to 180 degrees
- moved R19 2.33 mm to (1.14, -67.3), turned to 180 degrees
- moved C24 2.10 mm to (3.17, -66.2), turned to 180 degrees
- moved R18 2.10 mm to (3.17, -67.3), turned to 0 degrees
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Connections:
- C1 pad 1: VD -> +BATT
- C15 pad 1: VD -> +BATT
- C17 pad 1: VD -> +BATT
- C18 pad 1: VD -> +BATT
- C19 pad 1: VD -> +BATT
- C2 pad 1: +BATT -> /PWR3V_ON
- C23 pad 1: VD -> +BATT
- C4 pad 1: VD -> +BATT
- C5 pad 1: VD -> +BATT
- D4 pad 1: Net-(D4-K) -> /PWR3V_ON
- D4 pad 2: /WPS -> Net-(D4-A)
- J5 pad 10: unconnected-(J5-UIM_DATA-Pad10) -> /UIM_DATA
- J5 pad 12: unconnected-(J5-UIM_CLK-Pad12) -> /UIM_CLK
- J5 pad 14: unconnected-(J5-~{UIM_RESET}-Pad14) -> /UIM_RST
- J5 pad 16: unconnected-(J5-UIM_VPP-Pad16) -> /UIM_VPP
- J5 pad 17: unconnected-(J5-UIM_C8-Pad17) -> Net-(J5-UIM_C8)
- J5 pad 19: unconnected-(J5-UIM_C4-Pad19) -> Net-(J5-UIM_C4)
- J5 pad 3: unconnected-(J5-COEX1-Pad3) -> /UART1_CTS
- J5 pad 30: unconnected-(J5-SMB_CLK-Pad30) -> Net-(J5-SMB_CLK)
- J5 pad 32: unconnected-(J5-SMB_DATA-Pad32) -> Net-(J5-SMB_DATA)
- J5 pad 36: /USB1_DP -> /USB1_DM
- J5 pad 38: /USB1_DM -> /USB1_DP
- J5 pad 42: unconnected-(J5-~{LED_WWAN}-Pad42) -> Net-(J5-~{LED_WWAN})
- J5 pad 45: Net-(J5-Reserved-Pad45) -> /UART1_RXD
- J5 pad 46: unconnected-(J5-~{LED_WPAN}-Pad46) -> Net-(J5-~{LED_WPAN})
- J5 pad 5: unconnected-(J5-COEX2-Pad5) -> /UART1_RTS
- J5 pad 51: Net-(J5-Reserved-Pad51) -> /UART1_TXD
- J5 pad 8: unconnected-(J5-UIM_PWR-Pad8) -> /UIM_PWR
- J6 pad 1: /UART0_TXD -> /UIM_PWR
- J6 pad 2: /UART0_RXD -> /UIM_RST
- J6 pad 3: /UART1_TXD -> /UIM_CLK
- J6 pad 5: /UART1_RTS -> -BATT
- J6 pad 6: /UART1_CTS -> /UIM_VPP
- J6 pad 7: -BATT -> /UIM_DATA
- J7 pad 5: Net-(J7-Pin_5) -> /UART0_TXD
- J7 pad 6: Net-(J7-Pin_6) -> /UART0_RXD
- Q3 pad 1: Net-(Q3-G) -> Net-(D4-A)
- Q3 pad 3: Net-(D4-K) -> /WPS
- R1 pad 1: Net-(U3-EN) -> /PWR5V_ON
- R1 pad 2: Net-(U3-VINA) -> Net-(U3-EN)
- R4 pad 1: +BATT -> Net-(U3-EN)
- R4 pad 2: Net-(D4-K) -> -BATT
- R5 pad 1: /POWER_LED -> /PWR3V_ON
- R5 pad 2: Net-(Q3-G) -> Net-(U4-EN)
- R7 pad 1: Net-(U4-EN) -> Net-(D4-A)
- R7 pad 2: Net-(U4-VINA) -> Net-(R7-Pad2)
- R90 pad 2: Net-(J7-Pin_5) -> Net-(J7-Pin_7)
- R97 pad 1: Net-(J7-Pin_7) -> Net-(J7-Pin_9)
- SW2 pad 1: -BATT -> Net-(R7-Pad2)
- SW2 pad 2: Net-(D4-K) -> +BATT
- TP17 pad 1: Net-(J5-Reserved-Pad45) -> Net-(J5-UIM_C4)
- TP18 pad 1: Net-(J5-Reserved-Pad51) -> Net-(J5-UIM_C8)
- TP19 pad 1: Net-(D4-K) -> /PWR3V_ON
- U2 pad F17: Net-(J7-Pin_5) -> Net-(J7-Pin_7)
- U2 pad G16: Net-(J7-Pin_6) -> Net-(J7-Pin_8)
- U2 pad G18: Net-(J7-Pin_8) -> Net-(J7-Pin_10)
- U2 pad R17: unconnected-(U2E-GE2_RXCLK-PadR17) -> Net-(U2E-GE2_RXCLK)
- U2 pad T16: unconnected-(U2E-GE2_RXDV-PadT16) -> Net-(U2E-GE2_RXDV)
- U2 pad T17: unconnected-(U2E-GE2_RXD0-PadT17) -> Net-(U2E-GE2_RXD0)
- U2 pad T18: unconnected-(U2E-GE2_RXD1-PadT18) -> /PB_INT
- U2 pad U15: unconnected-(U2E-MDIO-PadU15) -> Net-(U2E-MDIO)
- U2 pad U16: unconnected-(U2E-GE2_RXD2-PadU16) -> /PWR5V_ON
- U2 pad U17: unconnected-(U2E-GE2_RXD3-PadU17) -> /PWR_ON
- U2 pad V16: /EN_DC -> /Y3-
- U2 pad V18: /PB_INT -> /Y4-
- U2 pad W17: /Y2- -> /G4-
- U2 pad W18: /POWER_LED -> /Y2-
- U2 pad Y17: /Y0- -> /G2-
- U2 pad Y18: /Y1- -> /G3-
- U3 pad 10: VD -> +BATT
- U3 pad 11: VD -> +BATT
- U3 pad 14: unconnected-(U3-PG-Pad14) -> /D2DB_PORST_N
- U4 pad 10: VD -> +BATT
- U4 pad 11: VD -> +BATT

Commit message: update pcb
Parts:
- removed R97: 22R, Resistor_SMD:R_0402_1005Metric
- C115, C130, C131, C132, C196, R12, R161, R4, R62, R63, R64, R65, R66, R67, R7, R86, TP19: moved to B.Cu
- C194, D3, R128, R5, TP20, TP21: moved to F.Cu
- moved FID1 84.1 mm to (49.0, -82.0)
- moved FID4 60.9 mm to (3.00, -24.0)
- moved FID5 45.8 mm to (54.0, -24.0)
- moved FID3 37.5 mm to (50.0, -3.00)
- moved R93 35.6 mm to (51.7, -56.0), turned to 180 degrees
- moved R94 34.9 mm to (51.7, -58.4)
- moved D2 34.3 mm to (53.1, -53.5), turned to 180 degrees
- moved R4 34.2 mm to (2.41, -73.9), turned to 180 degrees
- moved C142 29.5 mm to (44.8, -75.7)
- moved C138 28.5 mm to (44.8, -74.7)
- moved R17 28.1 mm to (20.8, -58.0)
- moved C133 28.0 mm to (44.8, -76.7)
- moved C137 27.8 mm to (44.8, -73.7)
- moved R7 24.0 mm to (31.0, -88.4), turned to -90 degrees
- moved J6 21.4 mm to (45.5, -86.7), turned to 90 degrees
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Connections:
- U2 pad G17: Net-(U2B-JTDO) -> Net-(J7-Pin_9)
