File: hardware/ethernet.kicad_sch (KiCad schematic)
At the start: 71 parts, among them J1 DS1128-09-S8B8X, J2 DS1128-09-S8B8X, J3 DS1128-09-S8B8X, U2 MT7621A

Commit message: update cap and dru
Parts:
- removed C103, C81, C82, C85: 4.7u, Capacitor_SMD:C_0805_2012Metric, symbol Device:C_Small
- added C52 (x4): 4.7u, Capacitor_SMD:C_0603_1608Metric, symbol Device:C_Small
- C100, C101, C102, C104, C106, C109, C110, C78, C79, C80, C83, C84, C86, C87, C88, C89, C90, C91, C92, C93, C94, C95, C96, C97, C98, C99: footprint Capacitor_SMD:C_0603_1608Metric -> Capacitor_SMD:C_0402_1005Metric; lcsc C14663 -> C307331
- C105, C107, C108: Voltage 1Kv -> 1kV
- R44, R45: footprint Resistor_SMD:R_0603_1608Metric -> Resistor_SMD:R_0402_1005Metric; lcsc C21190 -> C11702
- R46, R49: footprint Resistor_SMD:R_0603_1608Metric -> Resistor_SMD:R_0402_1005Metric
- R47: footprint Resistor_SMD:R_0603_1608Metric -> Resistor_SMD:R_0402_1005Metric; lcsc C23352 -> C25769
- R48: footprint Resistor_SMD:R_0603_1608Metric -> Resistor_SMD:R_0402_1005Metric; lcsc C23162 -> C25900
- R50, R51, R52, R53, R54, R55, R56, R57, R58, R59, R60, R61: footprint Resistor_SMD:R_0603_1608Metric -> Resistor_SMD:R_0402_1005Metric; lcsc C4275 -> C25133
- R62, R63, R64, R65, R66, R67: footprint Resistor_SMD:R_0603_1608Metric -> Resistor_SMD:R_0402_1005Metric; lcsc C23138 -> C25104
- TP10, TP11, TP12, TP13, TP14: value TestPoint -> TP
Connections:
- net +1V0: now also C52.1, C52.1, C52.1
- net +3V3: now also C52.1
- net ESW_TXVN_A_P2: now also TR1.11 (TD4+); no longer TR3.11 (TD4+)
- net ESW_TXVN_B_P2: now also TR1.7 (CT); no longer TR3.7 (CT)
- net ESW_TXVN_C_P2: now also TR1.5 (TD2+); no longer TR3.5 (TD2+)
- net ESW_TXVN_D_P2: now also TR1.1 (CT); no longer TR3.1 (CT)
- net ESW_TXVP_A_P2: now also TR1.12 (TD4-); no longer TR3.12 (TD4-)
- net ESW_TXVP_B_P2: now also TR1.8 (TD3+); no longer TR3.8 (TD3+)
- net ESW_TXVP_C_P2: now also TR1.6 (TD2-); no longer TR3.6 (TD2-)
- net ESW_TXVP_D_P2: now also TR1.2 (TD1+); no longer TR3.2 (TD1+)
- net G2-: now also J1.9
- net GND: now also C52.2
- net Y0-: no longer J1.11
- net Y1-: no longer J2.11, J3.11
- net Y2-: now also J1.11
- net P3A_P: now reaches J2.1, TR2.13 (MX4-)
- net P3A_N: now reaches J2.2, TR2.14 (MX4+)
- net P3B_P: now reaches J2.3, TR2.17 (MX3+)
- net P3C_P: now reaches J2.4, TR2.19 (MX2-)
- net P3C_N: now reaches J2.5, TR2.20 (MX2+)
- net P3B_N: now reaches J2.6, TR2.18 (CT)
- net P3D_P: now reaches J2.7, TR2.23 (MX1+)
- net P3D_N: now reaches J2.8, TR2.24 (CT)
- net P4A_P: now reaches J1.1, TR1.13 (MX4-)
- net P4A_N: now reaches J1.2, TR1.14 (MX4+)
- net P4B_P: now reaches J1.3, TR1.17 (MX3+)
- net P4C_P: now reaches J1.4, TR1.19 (MX2-)
- net P4C_N: now reaches J1.5, TR1.20 (MX2+)
- net P4B_N: now reaches J1.6, TR1.18 (CT)
- net P4D_P: now reaches J1.7, TR1.23 (MX1+)
- net P4D_N: now reaches J1.8, TR1.24 (CT)
- net at C102.2, C104.2, C106.2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: now also C52.2, C52.2, C52.2
- net P2A_P: now reaches J3.1, TR3.13 (MX4-)
- net P2A_N: now reaches J3.2, TR3.14 (MX4+)
- net P2B_P: now reaches J3.3, TR3.17 (MX3+)
- net P2C_P: now reaches J3.4, TR3.19 (MX2-)
- net P2C_N: now reaches J3.5, TR3.20 (MX2+)
- net P2B_N: now reaches J3.6, TR3.18 (CT)
- net P2D_P: now reaches J3.7, TR3.23 (MX1+)
- net P2D_N: now reaches J3.8, TR3.24 (CT)
- net ESW_TXVN_C_P3: now reaches U2.AA10 (ESW_TXVN_C_P3)
- net ESW_TXVN_C_P3: now also TR2.5 (TD2+)
- net ESW_TXVP_A_P4: now reaches U2.AA11 (ESW_TXVP_A_P4)
- net ESW_TXVP_A_P4: now also TR3.12 (TD4-)
- net ESW_TXVP_C_P4: now reaches U2.AA13 (ESW_TXVP_C_P4)
- net ESW_TXVP_C_P4: now also TR3.6 (TD2-)
- net ESW_TXVP_D_P3: now reaches U2.V10 (ESW_TXVP_D_P3)
- net ESW_TXVP_D_P3: now also TR2.2 (TD1+)
- net ESW_TXVN_D_P3: now reaches U2.W10 (ESW_TXVN_D_P3)
- net ESW_TXVN_D_P3: now also TR2.1 (CT)
- net ESW_TXVN_B_P4: now reaches U2.W12 (ESW_TXVN_B_P4)
- net ESW_TXVN_B_P4: now also TR3.7 (CT)
- net ESW_TXVP_D_P4: now reaches U2.W14 (ESW_TXVN_D_P4)
- net ESW_TXVP_D_P4: now also TR3.2 (TD1+)
- net ESW_TXVP_A_P3: now reaches U2.W8 (ESW_TXVP_A_P3)
- net ESW_TXVP_A_P3: now also TR2.12 (TD4-)
- net ESW_TXVP_B_P3: now reaches U2.W9 (ESW_TXVP_B_P3)
- net ESW_TXVP_B_P3: now also TR2.8 (TD3+)
- net ESW_TXVP_C_P3: now reaches U2.Y10 (ESW_TXVP_C_P3)
- net ESW_TXVP_C_P3: now also TR2.6 (TD2-)
- net ESW_TXVN_A_P4: now reaches U2.Y11 (ESW_TXVN_A_P4)
- net ESW_TXVN_A_P4: now also TR3.11 (TD4+)
- net ESW_TXVP_B_P4: now reaches U2.Y12 (ESW_TXVP_B_P4)
- net ESW_TXVP_B_P4: now also TR3.8 (TD3+)
- net ESW_TXVN_C_P4: now reaches U2.Y13 (ESW_TXVN_C_P4)
- net ESW_TXVN_C_P4: now also TR3.5 (TD2+)
- net ESW_TXVN_D_P4: now reaches U2.Y14 (ESW_TXVP_D_P4)
- net ESW_TXVN_D_P4: now also TR3.1 (CT)
- net ESW_TXVN_A_P3: now reaches U2.Y8 (ESW_TXVN_A_P3)
- net ESW_TXVN_A_P3: now also TR2.11 (TD4+)
- net ESW_TXVN_B_P3: now reaches U2.Y9 (ESW_TXVN_B_P3)
- net ESW_TXVN_B_P3: now also TR2.7 (CT)
- net ESW_TXVN_A_P0: no longer names the net of U2.R5 (ESW_TXVN_A_P0)
- net ESW_TXVN_A_P0: no longer TR1.11 (TD4+)
- net ESW_TXVN_A_P1: no longer names the net of U2.U4 (ESW_TXVN_A_P1)
- net ESW_TXVN_A_P1: no longer TR2.11 (TD4+)
- net ESW_TXVN_B_P0: no longer names the net of U2.R3 (ESW_TXVN_B_P0)
- net ESW_TXVN_B_P0: no longer TR1.7 (CT)
- net ESW_TXVN_B_P1: no longer names the net of U2.V3 (ESW_TXVN_B_P1)
- net ESW_TXVN_B_P1: no longer TR2.7 (CT)
- net ESW_TXVN_C_P0: no longer names the net of U2.T3 (ESW_TXVN_C_P0)
- net ESW_TXVN_C_P0: no longer TR1.5 (TD2+)
- net ESW_TXVN_C_P1: no longer names the net of U2.W2 (ESW_TXVN_C_P1)
- net ESW_TXVN_C_P1: no longer TR2.5 (TD2+)
- net ESW_TXVN_D_P0: no longer names the net of U2.U2 (ESW_TXVN_D_P0)
- net ESW_TXVN_D_P0: no longer TR1.1 (CT)
- net ESW_TXVN_D_P1: no longer names the net of U2.Y2 (ESW_TXVN_D_P1)
- net ESW_TXVN_D_P1: no longer TR2.1 (CT)
- net ESW_TXVP_A_P0: no longer names the net of U2.T5 (ESW_TXVP_A_P0)
- net ESW_TXVP_A_P0: no longer TR1.12 (TD4-)
- net ESW_TXVP_A_P1: no longer names the net of U2.T4 (ESW_TXVP_A_P1)
- net ESW_TXVP_A_P1: no longer TR2.12 (TD4-)
- net ESW_TXVP_B_P0: no longer names the net of U2.R2 (ESW_TXVP_B_P0)
- net ESW_TXVP_B_P0: no longer TR1.8 (TD3+)
- net ESW_TXVP_B_P1: no longer names the net of U2.V2 (ESW_TXVP_B_P1)
- net ESW_TXVP_B_P1: no longer TR2.8 (TD3+)
- net ESW_TXVP_C_P0: no longer names the net of U2.T2 (ESW_TXVP_C_P0)
- net ESW_TXVP_C_P0: no longer TR1.6 (TD2-)
- net ESW_TXVP_C_P1: no longer names the net of U2.W1 (ESW_TXVP_C_P1)
- net ESW_TXVP_C_P1: no longer TR2.6 (TD2-)
- net ESW_TXVP_D_P0: no longer names the net of U2.U1 (ESW_TXVP_D_P0)
- net ESW_TXVP_D_P0: no longer TR1.2 (TD1+)
- net ESW_TXVP_D_P1: no longer names the net of U2.Y1 (ESW_TXVP_D_P1)
- net ESW_TXVP_D_P1: no longer TR2.2 (TD1+)
- net G0- renamed P0_LED_0
- net P0_LED_0: no longer J1.9
- removed net G1-: J2.9, J3.9, U2.Y16 (ESW_P1_LED_0)
- net P3_LED_0 renamed G3-
- net G3-: now also J2.9
- net P4_LED_0 renamed G4-
- net G4-: now also J3.9
- new net P1_LED_0: U2.Y16 (ESW_P1_LED_0)
- new net Y3-: J2.11
- new net Y4-: J3.11
- no-connect marks 23 -> 7
Other:
- moved on the sheet: C87

Commit message: update pcb
Parts:
- TP10, TP11, TP12, TP13, TP14: footprint TestPoint:TestPoint_Pad_D1.0mm -> MAS_Package_std:TestPoint_Pad_D1mm
Changed lines of the file:
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@@
       (effects (font (size 1.27 1.27)) (justify left) hide)
     )
-    (property "Footprint" "TestPoint:TestPoint_Pad_D1.0mm" (at 205.74 142.24 0)
+    (property "Footprint" "MAS_Package_std:TestPoint_Pad_D1mm" (at 205.74 142.24 0)
       (effects (font (size 1.27 1.27)) hide)
     )
@@
       (effects (font (size 1.27 1.27)) (justify left) hide)
     )
-    (property "Footprint" "TestPoint:TestPoint_Pad_D1.0mm" (at 133.35 142.24 0)
+    (property "Footprint" "MAS_Package_std:TestPoint_Pad_D1mm" (at 133.35 142.24 0)
       (effects (font (size 1.27 1.27)) hide)
     )
@@
       (effects (font (size 1.27 1.27)) (justify left) hide)
     )
-    (property "Footprint" "TestPoint:TestPoint_Pad_D1.0mm" (at 147.32 116.84 0)
+    (property "Footprint" "MAS_Package_std:TestPoint_Pad_D1mm" (at 147.32 116.84 0)
       (effects (font (size 1.27 1.27)) hide)
     )
@@
       (effects (font (size 1.27 1.27)) (justify left) hide)
     )
-    (property "Footprint" "TestPoint:TestPoint_Pad_D1.0mm" (at 147.32 144.78 0)
+    (property "Footprint" "MAS_Package_std:TestPoint_Pad_D1mm" (at 147.32 144.78 0)
       (effects (font (size 1.27 1.27)) hide)
     )
@@
       (effects (font (size 1.27 1.27)) (justify left) hide)
     )
-    (property "Footprint" "TestPoint:TestPoint_Pad_D1.0mm" (at 205.74 144.78 0)
-      (effects (font (size 1.27 1.27)) hide)
-    )
+    (property "Footprint" "MAS_Package_std:TestPoint_Pad_D1mm" (at 205.74 144.78 0)
+      (effects (font (size 1.27 1.27)) hide)
+    )
