File: hardware/interface.kicad_sch (KiCad schematic)
At the start: 68 parts, among them J6 IDC-08M, J7 IDC-08M, J8 USB_C_Receptacle, U12 TPD2EUSB30, U13 TPD2EUSB30, U14 TPD2EUSB30, U2 MT7621A, Y1 X322540MPB4SI

Commit message: update pcb
Connections:
- net PCIE_CK0_N: now also TP26.1
- net PCIE_CK0_P: now also TP25.1
- net PCIE_CK1_N: no longer TP26.1
- net PCIE_CK1_P: no longer TP25.1
- net PCIE_RX0_N: now also TP30.1
- net PCIE_RX0_P: now also TP29.1
- net PCIE_RX1_N: no longer TP30.1
- net PCIE_RX1_P: no longer TP29.1
- net PCIE_TX0_N: now also TP28.1
- net PCIE_TX0_P: now also TP27.1
- net PCIE_TX1_N: no longer TP28.1
- net PCIE_TX1_P: no longer TP27.1
Other:
- moved on the sheet: TP25, TP26, TP27, TP28, TP29, TP30

Commit message: update cap and dru
Parts:
- removed C158: 10u, Capacitor_SMD:C_0805_2012Metric, symbol Device:C_Small
- removed C163, C176, C177, C179: 470n, Capacitor_SMD:C_0603_1608Metric, symbol Device:C_Small
- removed TP25, TP26, TP27, TP28, TP29, TP30: TestPoint, TestPoint:TestPoint_Pad_D1.0mm, symbol Connector:TestPoint
- added C52 (x4): 470n, Capacitor_SMD:C_0402_1005Metric, symbol Device:C_Small
- added C52: 4.7u, Capacitor_SMD:C_0603_1608Metric, symbol Device:C_Small
- C159, C160, C161, C162, C164, C165, C166, C167, C168, C169, C170, C171, C172, C173, C178: footprint Capacitor_SMD:C_0603_1608Metric -> Capacitor_SMD:C_0402_1005Metric; lcsc C14663 -> C307331
- C174, C175: footprint Capacitor_SMD:C_0603_1608Metric -> Capacitor_SMD:C_0402_1005Metric; lcsc C1647 -> C1549
- R100, R103: footprint Resistor_SMD:R_0603_1608Metric -> Resistor_SMD:R_0402_1005Metric; lcsc C23352 -> C25769
- R101, R102: footprint Resistor_SMD:R_0603_1608Metric -> Resistor_SMD:R_0402_1005Metric; lcsc C31850 -> C25768
- R104, R105, R106, R107, R108, R113, R114, R98, R99: footprint Resistor_SMD:R_0603_1608Metric -> Resistor_SMD:R_0402_1005Metric; lcsc C21189 -> C17168
- R109, R110, R111, R112: footprint Resistor_SMD:R_0603_1608Metric -> Resistor_SMD:R_0402_1005Metric; lcsc C23197 -> C25125
- R90: footprint Resistor_SMD:R_0603_1608Metric -> Resistor_SMD:R_0402_1005Metric; lcsc C21190 -> C11702
- R91, R92, R93, R94, R95, R96, R97: footprint Resistor_SMD:R_0603_1608Metric -> Resistor_SMD:R_0402_1005Metric; lcsc C23345 -> C25092
- TP19, TP20, TP21, TP22, TP23, TP24: value TestPoint -> TP
Connections:
- net +3V3: now also C52.2
- net +5V: now also C52.1
- net GND: now also C52.1, C52.1, C52.1, C52.2, C52.2
- net at C168.1, R108.2, U2.K4 (AVDD33_SSUSB)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: now also C52.1
- net at C178.2, R113.2, U2.J1 (AVDD12_SSUSB): now also C52.2
- net at C169.2, R114.2, U2.J18 (AVDD12_PE): now also C52.2
- no-connect marks 2 -> 4

Commit message: pinlayout for pci-e
Parts:
- added C111, C112, C113, C114, C117, C118, C121, C122: 100n, Capacitor_SMD:C_0402_1005Metric, symbol Device:C_Small
- added C52 (x6): 10u, Capacitor_SMD:C_0603_1608Metric, symbol Device:C_Small
- added D1: LEDY, Diode_SMD:D_0603_1608Metric, symbol Device:LED_Small
- added J10: AS0BC21-S30BM-7H, MAS_Package_std:Bus_M.2_Socket_M, symbol Connector:Bus_M.2_Socket_M
- added J5: miniPCI-E_52P_5.2, MAS_Package_std:BUS_PCI_Express_Mini_Dual, symbol Connector:Bus_PCI_Express_Mini
- added R116: 1k, Resistor_SMD:R_0402_1005Metric, symbol Device:R_Small
- added R3 (x3), R69, R70: 0R, Resistor_SMD:R_0402_1005Metric, symbol Device:R_Small
- added R68, R71: 51R, Resistor_SMD:R_0402_1005Metric, symbol Device:R_Small
- added R87 (x2): 4.7k, Resistor_SMD:R_0402_1005Metric, symbol Device:R_Small
- added TP15, TP16, TP17, TP18, TP25, TP26, TP27, TP28, TP29, TP30: TP, TestPoint:TestPoint_Pad_D1.0mm, symbol Connector:TestPoint
Connections:
- net +3V3: now also C117.1, C122.1, C52.1, C52.1, C52.1, C52.1, J10.12 (3.3V), J10.14 (3.3V), J10.16 (3.3V), J10.18 (3.3V), J10.2 (3.3V), J10.4 (3.3V), J10.70 (3.3V), J10.72 (3.3V), J10.74 (3.3V), J5.2 (+3V3AUX), J5.24 (+3V3AUX), J5.39 (+3V3AUX), J5.41 (+3V3AUX), J5.52 (+3V3AUX), R87.2, R87.2
- net +5V: now also R3.2
- net GND: now also C117.2, C118.2, C121.2, C122.2, C52.2, C52.2, C52.2, C52.2, C52.2, C52.2, J10.1 (GND), J10.15 (GND), J10.21 (GND), J10.27 (GND), J10.3 (GND), J10.33 (GND), J10.39 (GND), J10.45 (GND), J10.51 (GND), J10.57 (GND), J10.71 (GND), J10.73 (GND), J10.75 (GND), J10.9 (GND), J5.15 (GND), J5.18 (GND), J5.21 (GND), J5.26 (GND), J5.27 (GND), J5.29 (GND), J5.34 (GND), J5.35 (GND), J5.37 (GND), J5.4 (GND), J5.40 (GND), J5.43 (GND), J5.50 (GND), J5.9 (GND), J5.MP, R116.1, R68.2, R71.2
- net PCIE_CK0_N: now also R105.1, R110.1, J5.11 (REFCLK-); no longer R107.1, R112.1
- net PCIE_CK0_P: now also R104.1, R109.1, J5.13 (REFCLK+); no longer R106.1, R111.1
- net PCIE_CK1_N: now also R107.1, R112.1, J10.53 (REFCLKn); no longer R105.1, R110.1
- net PCIE_CK1_P: now also R106.1, R111.1, J10.55 (REFCLKp); no longer R104.1, R109.1
- net PCIE_RX0_N: now also C171.2, J5.23 (PERn0); no longer C173.2
- net PCIE_RX0_P: now also C170.2, J5.25 (PERp0); no longer C172.2
- net PCIE_RX1_N: now also C173.2, J10.41 (PERn0/SATA-B+); no longer C171.2
- net PCIE_RX1_P: now also C172.2, J10.43 (PERp0/SATA-B-); no longer C170.2
- net PCIE_TX0_N: now also C165.2, J5.31 (PETn0); no longer C167.2
- net PCIE_TX0_P: now also C164.2, J5.33 (PETp0); no longer C166.2
- net PCIE_TX1_N: now also C167.2, J10.47 (PETn0/SATA-A-); no longer C165.2
- net PCIE_TX1_P: now also C166.2, J10.49 (PETp0/SATA-A+); no longer C164.2
- net PERST_N: now also R3.1, R3.1
- net USB1_DM: now reaches U2.K1 (USB_DM_P1)
- net USB1_DM: now also J5.38 (USB_D+)
- net USB1_DP: now reaches U2.K2 (USB_DP_P1)
- net USB1_DP: now also J5.36 (USB_D-)
- net at U2.M13 (PCIE_CKP2): now also R69.2
- net at U2.M14 (PCIE_CKN2): now also R70.2
- net at U2.M17 (PCIE_RXP2): now also C113.1
- net at U2.M18 (PCIE_RXN2): now also C114.1
- net at U2.N16 (PCIE_TXP2): now also C111.1
- net at U2.N17 (PCIE_TXN2): now also C112.1
- new net: D1.1 (K), R116.2
- new net: C121.1, C52.1, J5.47 (Reserved), J5.49 (Reserved), R3.1
- new net: J10.52 (~{CLKREQ}), TP26.1
- new net: D1.2 (A), J5.44 (~{LED_WLAN})
- new net: J5.1 (~{WAKE}), TP25.1
- new net: J5.20 (~{W_DISABLE}), TP16.1
- new net: J5.22 (~{PERST}), R3.2, R87.1
- new net: J5.45 (Reserved), TP17.1
- new net: J5.51 (Reserved), TP18.1
- new net: J5.7 (~{CLKREQ}), TP15.1
- new net: J10.50 (~{PERST}), R3.2, R87.1
- new net: J10.10 (DAS/~{DSS}/~{LED1}), TP30.1
- new net: J10.54 (~{PEWAKE}), TP27.1
- new net +1V5: C118.1, C52.1, J5.28 (+1V5), J5.48 (+1V5), J5.6 (+1V5)
- new net PCIE_CK2_N: R70.1, R71.1, TP29.1
- new net PCIE_CK2_P: R68.1, R69.1, TP28.1
- new net PCIE_RX2_N: C114.2, J10.29 (PERn1)
- new net PCIE_RX2_P: C113.2, J10.31 (PERp1)
- new net PCIE_TX2_N: C112.2, J10.35 (PETn1)
- new net PCIE_TX2_P: C111.2, J10.37 (PETp1)
- no-connect marks 4 -> 26

Commit message: update pcb
Parts:
- TP15, TP16, TP17, TP18, TP19, TP20, TP21, TP22, TP23, TP24, TP25, TP26, TP27, TP28, TP29, TP30: footprint TestPoint:TestPoint_Pad_D1.0mm -> MAS_Package_std:TestPoint_Pad_D1mm
Changed lines of the file:
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@@
       (effects (font (size 1.27 1.27)) (justify left) hide)
     )
-    (property "Footprint" "TestPoint:TestPoint_Pad_D1.0mm" (at 147.32 87.63 0)
+    (property "Footprint" "MAS_Package_std:TestPoint_Pad_D1mm" (at 147.32 87.63 0)
       (effects (font (size 1.27 1.27)) hide)
     )
@@
       (effects (font (size 1.27 1.27)) (justify left) hide)
     )
-    (property "Footprint" "TestPoint:TestPoint_Pad_D1.0mm" (at -36.83 -33.02 0)
+    (property "Footprint" "MAS_Package_std:TestPoint_Pad_D1mm" (at -36.83 -33.02 0)
       (effects (font (size 1.27 1.27)) hide)
     )
@@
       (effects (font (size 1.27 1.27)) (justify left) hide)
     )
-    (property "Footprint" "TestPoint:TestPoint_Pad_D1.0mm" (at -86.36 -76.2 0)
+    (property "Footprint" "MAS_Package_std:TestPoint_Pad_D1mm" (at -86.36 -76.2 0)
       (effects (font (size 1.27 1.27)) hide)
     )
@@
       (effects (font (size 1.27 1.27)) (justify left) hide)
     )
-    (property "Footprint" "TestPoint:TestPoint_Pad_D1.0mm" (at -45.72 -101.6 0)
+    (property "Footprint" "MAS_Package_std:TestPoint_Pad_D1mm" (at -45.72 -101.6 0)
       (effects (font (size 1.27 1.27)) hide)
     )
@@
       (effects (font (size 1.27 1.27)) (justify left) hide)
     )
-    (property "Footprint" "TestPoint:TestPoint_Pad_D1.0mm" (at -86.36 -81.28 0)
+    (property "Footprint" "MAS_Package_std:TestPoint_Pad_D1mm" (at -86.36 -81.28 0)
       (effects (font (size 1.27 1.27)) hide)
     )
@@
       (effects (font (size 1.27 1.27)) (justify left) hide)
     )
-    (property "Footprint" "TestPoint:TestPoint_Pad_D1.0mm" (at -86.36 -78.74 0)
+    (property "Footprint" "MAS_Package_std:TestPoint_Pad_D1mm" (at -86.36 -78.74 0)
       (effects (font (size 1.27 1.27)) hide)
     )
@@
       (effects (font (size 1.27 1.27)) (justify left) hide)
     )
-    (property "Footprint" "TestPoint:TestPoint_Pad_D1.0mm" (at 147.32 90.17 0)
+    (property "Footprint" "MAS_Package_std:TestPoint_Pad_D1mm" (at 147.32 90.17 0)
       (effects (font (size 1.27 1.27)) hide)
     )
@@
       (effects (font (size 1.27 1.27)) (justify left) hide)
     )
-    (property "Footprint" "TestPoint:TestPoint_Pad_D1.0mm" (at 139.7 67.31 0)
+    (property "Footprint" "MAS_Package_std:TestPoint_Pad_D1mm" (at 139.7 67.31 0)
       (effects (font (size 1.27 1.27)) hide)
     )
@@
       (effects (font (size 1.27 1.27)) (justify left) hide)
     )
-    (property "Footprint" "TestPoint:TestPoint_Pad_D1.0mm" (at 34.29 17.78 0)
+    (property "Footprint" "MAS_Package_std:TestPoint_Pad_D1mm" (at 34.29 17.78 0)
       (effects (font (size 1.27 1.27)) hide)
     )
@@
       (effects (font (size 1.27 1.27)) (justify left) hide)
     )
-    (property "Footprint" "TestPoint:TestPoint_Pad_D1.0mm" (at 139.7 59.69 0)
+    (property "Footprint" "MAS_Package_std:TestPoint_Pad_D1mm" (at 139.7 59.69 0)
       (effects (font (size 1.27 1.27)) hide)
     )
@@
       (effects (font (size 1.27 1.27)) (justify left) hide)
     )
-    (property "Footprint" "TestPoint:TestPoint_Pad_D1.0mm" (at -36.83 -30.48 0)
+    (property "Footprint" "MAS_Package_std:TestPoint_Pad_D1mm" (at -36.83 -30.48 0)
       (effects (font (size 1.27 1.27)) hide)
     )
@@
       (effects (font (size 1.27 1.27)) (justify left) hide)
     )
-    (property "Footprint" "TestPoint:TestPoint_Pad_D1.0mm" (at -35.56 25.4 0)
+    (property "Footprint" "MAS_Package_std:TestPoint_Pad_D1mm" (at -35.56 25.4 0)
       (effects (font (size 1.27 1.27)) hide)
     )
@@
       (effects (font (size 1.27 1.27)) (justify left) hide)
     )
-    (property "Footprint" "TestPoint:TestPoint_Pad_D1.0mm" (at -35.56 22.86 0)
+    (property "Footprint" "MAS_Package_std:TestPoint_Pad_D1mm" (at -35.56 22.86 0)
       (effects (font (size 1.27 1.27)) hide)
     )
@@
       (effects (font (size 1.27 1.27)) (justify left) hide)
     )
-    (property "Footprint" "TestPoint:TestPoint_Pad_D1.0mm" (at 139.7 62.23 0)
+    (property "Footprint" "MAS_Package_std:TestPoint_Pad_D1mm" (at 139.7 62.23 0)
       (effects (font (size 1.27 1.27)) hide)
     )
@@
       (effects (font (size 1.27 1.27)) (justify left) hide)
     )
-    (property "Footprint" "TestPoint:TestPoint_Pad_D1.0mm" (at 139.7 64.77 0)
+    (property "Footprint" "MAS_Package_std:TestPoint_Pad_D1mm" (at 139.7 64.77 0)
       (effects (font (size 1.27 1.27)) hide)
     )
@@
       (effects (font (size 1.27 1.27)) (justify left) hide)
     )
-    (property "Footprint" "TestPoint:TestPoint_Pad_D1.0mm" (at -45.72 -93.98 0)
+    (property "Footprint" "MAS_Package_std:TestPoint_Pad_D1mm" (at -45.72 -93.98 0)
       (effects (font (size 1.27 1.27)) hide)
     )
