File: hardware/memory.kicad_sch (KiCad schematic)
At the start: 49 parts, among them U10 W25Q256FVEIG, U2 MT7621A, U9 NT5CB64M16FP-DH (!)

Commit message: update cap and dru
Parts:
- removed C75, C76: 4.7u, Capacitor_SMD:C_0805_2012Metric, symbol Device:C_Small
- added C52 (x2): 4.7u, Capacitor_SMD:C_0603_1608Metric, symbol Device:C_Small
- C57, C58, C59, C60, C61, C62, C63, C64, C65, C66, C67, C68, C69, C70, C71, C72, C73, C74, C77: footprint Capacitor_SMD:C_0603_1608Metric -> Capacitor_SMD:C_0402_1005Metric; lcsc C14663 -> C307331
- R10, R11, R13, R14, R15, R20: footprint Resistor_SMD:R_0603_1608Metric -> Resistor_SMD:R_0402_1005Metric; lcsc C21190 -> C11702
- R2, R35: footprint Resistor_SMD:R_0603_1608Metric -> Resistor_SMD:R_0402_1005Metric; lcsc C23350 -> C114755
- R3: footprint Resistor_SMD:R_0603_1608Metric -> Resistor_SMD:R_0402_1005Metric; lcsc C21189 -> C17168
- R34: footprint Resistor_SMD:R_0603_1608Metric -> Resistor_SMD:R_0402_1005Metric; lcsc C22775 -> C153111
- R40, R41, R8: footprint Resistor_SMD:R_0603_1608Metric -> Resistor_SMD:R_0402_1005Metric
- R42, R43: footprint Resistor_SMD:R_0603_1608Metric -> Resistor_SMD:R_0402_1005Metric; lcsc C23162 -> C25900
- R9: footprint Resistor_SMD:R_0603_1608Metric -> Resistor_SMD:R_0402_1005Metric; lcsc C25804 -> C25744
- TP1, TP2, TP3, TP4, TP5, TP6, TP7, TP8, TP9: value TestPoint -> TP
Connections:
- net +1V5: now also C52.1, C52.1
- net GND: now also C52.2, C52.2

Commit message: add mini-pcie and m2
Parts:
- R40, R41: now not fitted; now left out of the parts list
Changed lines of the file:
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@@
   )
   (symbol (lib_id "Device:R_Small") (at 234.95 76.2 0) (mirror x) (unit 1)
-    (in_bom yes) (on_board yes) (dnp no)
+    (in_bom no) (on_board yes) (dnp yes)
     (property "Reference" "R40" (at 233.4514 75.0316 0)
       (effects (font (size 1.27 1.27)) (justify right))
@@
   )
   (symbol (lib_id "Device:R_Small") (at 237.49 48.26 0) (mirror x) (unit 1)
-    (in_bom yes) (on_board yes) (dnp no)
+    (in_bom no) (on_board yes) (dnp yes)
     (property "Reference" "R41" (at 235.9914 47.0916 0)
       (effects (font (size 1.27 1.27)) (justify right))

Commit message: update pcb
Parts:
- TP1, TP2, TP3, TP4, TP5, TP6, TP7, TP8, TP9: footprint TestPoint:TestPoint_Pad_D1.0mm -> MAS_Package_std:TestPoint_Pad_D1mm
Changed lines of the file:
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@@
       (effects (font (size 1.27 1.27)) (justify left) hide)
     )
-    (property "Footprint" "TestPoint:TestPoint_Pad_D1.0mm" (at -10.16 134.62 0)
+    (property "Footprint" "MAS_Package_std:TestPoint_Pad_D1mm" (at -10.16 134.62 0)
       (effects (font (size 1.27 1.27)) hide)
     )
@@
       (effects (font (size 1.27 1.27)) (justify left) hide)
     )
-    (property "Footprint" "TestPoint:TestPoint_Pad_D1.0mm" (at -10.16 101.6 0)
+    (property "Footprint" "MAS_Package_std:TestPoint_Pad_D1mm" (at -10.16 101.6 0)
       (effects (font (size 1.27 1.27)) hide)
     )
@@
       (effects (font (size 1.27 1.27)) (justify left) hide)
     )
-    (property "Footprint" "TestPoint:TestPoint_Pad_D1.0mm" (at -10.16 139.7 0)
+    (property "Footprint" "MAS_Package_std:TestPoint_Pad_D1mm" (at -10.16 139.7 0)
       (effects (font (size 1.27 1.27)) hide)
     )
@@
       (effects (font (size 1.27 1.27)) (justify left) hide)
     )
-    (property "Footprint" "TestPoint:TestPoint_Pad_D1.0mm" (at -10.16 144.78 0)
+    (property "Footprint" "MAS_Package_std:TestPoint_Pad_D1mm" (at -10.16 144.78 0)
       (effects (font (size 1.27 1.27)) hide)
     )
@@
       (effects (font (size 1.27 1.27)) (justify left) hide)
     )
-    (property "Footprint" "TestPoint:TestPoint_Pad_D1.0mm" (at -10.16 129.54 0)
+    (property "Footprint" "MAS_Package_std:TestPoint_Pad_D1mm" (at -10.16 129.54 0)
       (effects (font (size 1.27 1.27)) hide)
     )
@@
       (effects (font (size 1.27 1.27)) (justify left) hide)
     )
-    (property "Footprint" "TestPoint:TestPoint_Pad_D1.0mm" (at -10.16 147.32 0)
+    (property "Footprint" "MAS_Package_std:TestPoint_Pad_D1mm" (at -10.16 147.32 0)
       (effects (font (size 1.27 1.27)) hide)
     )
@@
       (effects (font (size 1.27 1.27)) (justify left) hide)
     )
-    (property "Footprint" "TestPoint:TestPoint_Pad_D1.0mm" (at -10.16 124.46 0)
+    (property "Footprint" "MAS_Package_std:TestPoint_Pad_D1mm" (at -10.16 124.46 0)
       (effects (font (size 1.27 1.27)) hide)
     )
@@
       (effects (font (size 1.27 1.27)) (justify left) hide)
     )
-    (property "Footprint" "TestPoint:TestPoint_Pad_D1.0mm" (at -10.16 114.3 0)
+    (property "Footprint" "MAS_Package_std:TestPoint_Pad_D1mm" (at -10.16 114.3 0)
       (effects (font (size 1.27 1.27)) hide)
     )
@@
       (effects (font (size 1.27 1.27)) (justify left) hide)
     )
-    (property "Footprint" "TestPoint:TestPoint_Pad_D1.0mm" (at -10.16 142.24 0)
-      (effects (font (size 1.27 1.27)) hide)
-    )
+    (property "Footprint" "MAS_Package_std:TestPoint_Pad_D1mm" (at -10.16 142.24 0)
+      (effects (font (size 1.27 1.27)) hide)
+    )
