File: hardware/other.kicad_sch (KiCad schematic)
At the start: 69 parts, among them Q4 BC817, SW3 TS-1187A-B-A-B, SW4 TS-1187A-B-A-B, U16 N096-2864KSWEG01-H30

Commit message: update pcb
Parts:
- C195, C198, C199, C200, C201: footprint Capacitor_SMD:C_0805_2012Metric -> Capacitor_SMD:C_0603_1608Metric
Changed lines of the file:
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@@
       (effects (font (size 1.27 1.27)) (justify left))
     )
-    (property "Footprint" "Capacitor_SMD:C_0805_2012Metric" (id 2) (at 227.33 50.8 0)
+    (property "Footprint" "Capacitor_SMD:C_0603_1608Metric" (id 2) (at 227.33 50.8 0)
       (effects (font (size 1.27 1.27)) hide)
     )
@@
       (effects (font (size 1.27 1.27)) (justify left))
     )
-    (property "Footprint" "Capacitor_SMD:C_0805_2012Metric" (id 2) (at 199.39 57.15 0)
+    (property "Footprint" "Capacitor_SMD:C_0603_1608Metric" (id 2) (at 199.39 57.15 0)
       (effects (font (size 1.27 1.27)) hide)
     )
@@
       (effects (font (size 1.27 1.27)) (justify left) hide)
     )
-    (property "Footprint" "Capacitor_SMD:C_0805_2012Metric" (id 2) (at 227.33 63.5 0)
+    (property "Footprint" "Capacitor_SMD:C_0603_1608Metric" (id 2) (at 227.33 63.5 0)
       (effects (font (size 1.27 1.27)) hide)
     )
@@
       (effects (font (size 1.27 1.27)) (justify left) hide)
     )
-    (property "Footprint" "Capacitor_SMD:C_0805_2012Metric" (id 2) (at 227.33 68.58 0)
+    (property "Footprint" "Capacitor_SMD:C_0603_1608Metric" (id 2) (at 227.33 68.58 0)
       (effects (font (size 1.27 1.27)) hide)
     )
@@
       (effects (font (size 1.27 1.27)) (justify left) hide)
     )
-    (property "Footprint" "Capacitor_SMD:C_0805_2012Metric" (id 2) (at 227.33 55.88 0)
-      (effects (font (size 1.27 1.27)) hide)
-    )
+    (property "Footprint" "Capacitor_SMD:C_0603_1608Metric" (id 2) (at 227.33 55.88 0)
+      (effects (font (size 1.27 1.27)) hide)
+    )

Commit message: update pcb
Parts:
- R126: footprint Resistor_SMD:R_0805_2012Metric -> Resistor_SMD:R_0603_1608Metric; chipdip 9000079478 -> (none); lcsc C17710 -> C23179
Changed lines of the file:
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@@
       (effects (font (size 1.27 1.27)) (justify right))
     )
-    (property "Footprint" "Resistor_SMD:R_0805_2012Metric" (id 2) (at -53.34 53.34 0)
+    (property "Footprint" "Resistor_SMD:R_0603_1608Metric" (id 2) (at -53.34 53.34 0)
       (effects (font (size 1.27 1.27)) hide)
     )
@@
       (effects (font (size 1.27 1.27)) hide)
     )
-    (property "chipdip" "9000079478" (id 4) (at -53.34 53.34 0)
+    (property "chipdip" "" (id 4) (at -53.34 53.34 0)
       (effects (font (size 1.27 1.27)) hide)
     )
@@
       (effects (font (size 1.27 1.27)) hide)
     )
-    (property "lcsc" "C17710" (id 6) (at -53.34 53.34 0)
+    (property "lcsc" "C23179" (id 6) (at -53.34 53.34 0)
       (effects (font (size 1.27 1.27)) hide)
     )

Commit message: update cap and dru
Parts:
- removed C195, C198, C199, C200, C201: 1u, Capacitor_SMD:C_0603_1608Metric, symbol Device:C_Small
- removed C202, C203: 4.7u, Capacitor_SMD:C_0805_2012Metric, symbol Device:C_Small
- added C52 (x7): 4.7u, Capacitor_SMD:C_0603_1608Metric, symbol Device:C_Small
- C193, C194, C196, C197: footprint Capacitor_SMD:C_0603_1608Metric -> Capacitor_SMD:C_0402_1005Metric; lcsc C14663 -> C307331
- R125: footprint Resistor_SMD:R_0603_1608Metric -> Resistor_SMD:R_0402_1005Metric; lcsc C25804 -> C25744
- R126: footprint Resistor_SMD:R_0603_1608Metric -> Resistor_SMD:R_0402_1005Metric; lcsc C23179 -> C25117
- R127: footprint Resistor_SMD:R_0603_1608Metric -> Resistor_SMD:R_0402_1005Metric; lcsc C21190 -> C11702
- R128: footprint Resistor_SMD:R_0603_1608Metric -> Resistor_SMD:R_0402_1005Metric; lcsc C25803 -> C25741
- R129, R132, R133, R135, R138, R140, R142, R144, R145, R148, R149, R151, R153, R155, R158, R159, R163, R166, R167: footprint Resistor_SMD:R_0603_1608Metric -> Resistor_SMD:R_0402_1005Metric; lcsc C23162 -> C25900
- R130, R131, R134, R136, R137, R139, R141, R143, R146, R147, R150, R152, R154, R156, R157, R160, R162, R172: footprint Resistor_SMD:R_0603_1608Metric -> Resistor_SMD:R_0402_1005Metric
- R161, R165, R168, R169, R170, R171: footprint Resistor_SMD:R_0603_1608Metric -> Resistor_SMD:R_0402_1005Metric; lcsc C21189 -> C17168
- R164: footprint Resistor_SMD:R_0603_1608Metric -> Resistor_SMD:R_0402_1005Metric; lcsc C365224 -> C170371
- TP31, TP32, TP33, TP34: value TestPoint -> TP
Connections:
- net 3V3O: now also C52.1, C52.2, C52.2
- net GND: now also C52.1, C52.1, C52.2, C52.2, C52.2
- net at U16.28 (VDisplay): now also C52.1
- net at U16.3 (C2N): now also C52.1
- net at U16.2 (C2P): now also C52.2
- net at U16.27 (VCOMH): now also C52.1
- net at U16.4 (C1P): now also C52.2
- net at U16.5 (C1N): now also C52.1

Commit message: update pcb
Parts:
- removed C193: 100n, Capacitor_SMD:C_0402_1005Metric, symbol Device:C_Small
- removed D2: LEDG, Diode_SMD:D_0603_1608Metric, symbol Device:LED_Small
- removed Q4: BC817, Package_TO_SOT_SMD:SOT-23, symbol Transistor_BJT:BC817
- removed R125: 10k, Resistor_SMD:R_0402_1005Metric, symbol Device:R_Small
- removed R126: 470R, Resistor_SMD:R_0402_1005Metric, symbol Device:R_Small
- removed R127: 1k, Resistor_SMD:R_0402_1005Metric, symbol Device:R_Small
- removed SW3: TS-1187A-B-A-B, Button_Switch_SMD:SW_SPST_TL3342, symbol Switch:SW_Push
- TP31, TP32, TP33, TP34: footprint TestPoint:TestPoint_Pad_D1.0mm -> MAS_Package_std:TestPoint_Pad_D1mm
