File: hardware/power.kicad_sch (KiCad schematic)
At the start: 106 parts, among them Q2 SSM6J501NU, Q3 FDV301N, SW2 TS-1187A-B-A-B, U1 SN74LVC1G175, U2 MT7621A, U3 TPS63020, U4 TPS63020, U5 MT3420B, U6 MT3420B, U7 MT3420B, U8 MT3420B

Commit message: update pcb
Parts:
- R5: footprint Resistor_SMD:R_0805_2012Metric -> Resistor_SMD:R_0603_1608Metric; chipdip 9000079478 -> (none); lcsc C17710 -> C23179
Connections:
- net GND: now also SW2.1; no longer SW2.2
- net at C9.1, R12.1, U1.1 (CLK): now also SW2.2; no longer SW2.1
Changed lines of the file:
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@@
       (effects (font (size 1.27 1.27)) (justify right))
     )
-    (property "Footprint" "Resistor_SMD:R_0805_2012Metric" (id 2) (at 53.34 171.45 0)
+    (property "Footprint" "Resistor_SMD:R_0603_1608Metric" (id 2) (at 53.34 171.45 0)
       (effects (font (size 1.27 1.27)) hide)
     )
@@
       (effects (font (size 1.27 1.27)) hide)
     )
-    (property "chipdip" "9000079478" (id 4) (at 53.34 171.45 0)
+    (property "chipdip" "" (id 4) (at 53.34 171.45 0)
       (effects (font (size 1.27 1.27)) hide)
     )
@@
       (effects (font (size 1.27 1.27)) hide)
     )
-    (property "lcsc" "C17710" (id 6) (at 53.34 171.45 0)
+    (property "lcsc" "C23179" (id 6) (at 53.34 171.45 0)
       (effects (font (size 1.27 1.27)) hide)
     )
@@
     (pin "2")
   )
-  (symbol (lib_id "Switch:SW_Push") (at 87.63 181.61 270) (unit 1)
-    (in_bom yes) (on_board yes) (fields_autoplaced)
-    (property "Reference" "SW2" (id 0) (at 95.25 181.61 0))
-    (property "Value" "TS-1187A-B-A-B" (id 1) (at 92.71 181.61 0))
-    (property "Footprint" "Button_Switch_SMD:SW_SPST_TL3342" (id 2) (at 92.71 181.61 0)
-      (effects (font (size 1.27 1.27)) hide)
-    )
-    (property "Datasheet" "https://datasheet.lcsc.com/lcsc/2002271431_XKB-Connectivity-TS-1187A-B-A-B_C318884.pdf" (id 3) (at 92.71 181.61 0)
-      (effects (font (size 1.27 1.27)) hide)
-    )
-    (property "lcsc" "C318884" (id 4) (at 87.63 181.61 0)
-      (effects (font (size 1.27 1.27)) hide)
-    )
-    (pin "1")
-    (pin "2")
-  )
   (symbol (lib_id "Device:C_Small") (at 331.47 74.93 0) (unit 1)
     (in_bom yes) (on_board yes)
@@
       (effects (font (size 1.27 1.27)) hide)
     )
+    (pin "1")
+    (pin "2")
+  )
+  (symbol (lib_id "Switch:SW_Push") (at 87.63 181.61 270) (mirror x) (unit 1)
+    (in_bom yes) (on_board yes) (fields_autoplaced)
+    (property "Reference" "SW2" (id 0) (at 91.44 180.3399 90)
+      (effects (font (size 1.27 1.27)) (justify left))
+    )
+    (property "Value" "TS-1187A-B-A-B" (id 1) (at 91.44 182.8799 90)
+      (effects (font (size 1.27 1.27)) (justify left))
+    )
+    (property "Footprint" "Button_Switch_SMD:SW_SPST_TL3342" (id 2) (at 92.71 181.61 0)
+      (effects (font (size 1.27 1.27)) hide)
+    )
+    (property "Datasheet" "https://datasheet.lcsc.com/lcsc/2002271431_XKB-Connectivity-TS-1187A-B-A-B_C318884.pdf" (id 3) (at 92.71 181.61 0)
+      (effects (font (size 1.27 1.27)) hide)
+    )
+    (property "lcsc" "C318884" (id 4) (at 87.63 181.61 0)
+      (effects (font (size 1.27 1.27)) hide)
+    )

Commit message: update cap and dru
Parts:
- removed C1, C17, C23, C36, C37, C4, C45, C46, C47, C48, C5, C55, C56, C6, C7: 10u, Capacitor_SMD:C_0805_2012Metric, symbol Device:C_Small
- removed C14, C15, C30, C31, C32, C33: 2.2u, Capacitor_SMD:C_0805_2012Metric, symbol Device:C_Small
- added C52 (x15): 10u, Capacitor_SMD:C_0603_1608Metric, symbol Device:C_Small
- added C52 (x6): 4.7u, Capacitor_SMD:C_0603_1608Metric, symbol Device:C_Small
- C10, C11, C12, C13, C16, C18, C19, C2, C20, C21, C22, C26, C27, C28, C29, C3, C38, C39, C42, C43, C44, C49, C50, C53, C54, C8, C9: footprint Capacitor_SMD:C_0603_1608Metric -> Capacitor_SMD:C_0402_1005Metric; lcsc C14663 -> C307331
- C24, C25: footprint Capacitor_SMD:C_0603_1608Metric -> Capacitor_SMD:C_0402_1005Metric; lcsc C282071 -> C1569
- C40, C41, C51, C52: footprint Capacitor_SMD:C_0603_1608Metric -> Capacitor_SMD:C_0402_1005Metric; lcsc C1653 -> C1555
- JP2, JP3, JP4, JP5, JP6, JP7: value J_Boot -> JP; footprint Jumper:SolderJumper-2_P1.3mm_Open_Pad1.0x1.5mm -> MAS_Package_nostd:SolderJumper_Open_Pad0.5x0.8mm
- R1, R12, R16, R6, R7: footprint Resistor_SMD:R_0603_1608Metric -> Resistor_SMD:R_0402_1005Metric; lcsc C21190 -> C11702
- R17, R26, R27, R28, R30, R32, R33, R36, R37, R39: footprint Resistor_SMD:R_0603_1608Metric -> Resistor_SMD:R_0402_1005Metric; lcsc C25803 -> C25741
- R18, R4: footprint Resistor_SMD:R_0603_1608Metric -> Resistor_SMD:R_0402_1005Metric; lcsc C25804 -> C25744
- R19: footprint Resistor_SMD:R_0603_1608Metric -> Resistor_SMD:R_0402_1005Metric; lcsc C22764 -> C325543
- R21: footprint Resistor_SMD:R_0603_1608Metric -> Resistor_SMD:R_0402_1005Metric; lcsc C23137 -> C25778
- R22: footprint Resistor_SMD:R_0603_1608Metric -> Resistor_SMD:R_0402_1005Metric; lcsc C23196 -> C25794
- R23: footprint Resistor_SMD:R_0603_1608Metric -> Resistor_SMD:R_0402_1005Metric; lcsc C22975 -> C100608
- R24, R25: footprint Resistor_SMD:R_0603_1608Metric -> Resistor_SMD:R_0402_1005Metric; lcsc C23231 -> C36871
- R29: footprint Resistor_SMD:R_0603_1608Metric -> Resistor_SMD:R_0402_1005Metric; lcsc C25808 -> C25750
- R31, R38: footprint Resistor_SMD:R_0603_1608Metric -> Resistor_SMD:R_0402_1005Metric; lcsc C22807 -> C25755
- R5: footprint Resistor_SMD:R_0603_1608Metric -> Resistor_SMD:R_0402_1005Metric; lcsc C23179 -> C25117
Connections:
- net +1V0: now also C52.1
- net +1V1: now also C52.1
- net +1V5: now also C52.1
- net +3V3: now also C52.1, C52.1, C52.1, C52.1
- net GND: now also C52.2, C52.2, C52.2, C52.2, C52.2, C52.2, C52.2, C52.2, C52.2, C52.2, C52.2, C52.2, C52.2, C52.2, C52.2, C52.2, C52.2, C52.2, C52.2, C52.2, C52.2
- net VD: now also C52.1, C52.1, C52.1, C52.1, C52.1, C52.1
- net at C40.1, C43.1, JP4.2 (B)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: now also C52.1
- net at C52.1, C54.1, JP7.2 (B)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: now also C52.1
- net at C41.1, C44.1, JP5.2 (B)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: now also C52.1
- net at C28.1, C34.1, JP2.2 (B)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: now also C52.1, C52.1
- net at C51.1, C53.1, JP6.2 (B)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: now also C52.1
- net at C29.1, C35.1, JP3.2 (B)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: now also C52.1, C52.1
Other:
- moved on the sheet: C42

Commit message: add mini-pcie and m2
Parts:
- L4, L5, L6, L7: value SLO0530H2R2MTT -> LVS303015-2R2M; footprint MAS_Package_std:Power_inductor_SMD_0530 -> Inductor_SMD:L_Wuerth_MAPI-3015; lcsc C325962 -> C285837
Changed lines of the file:
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@@
       (effects (font (size 1.27 1.27)))
     )
-    (property "Value" "SLO0530H2R2MTT" (at 214.63 68.58 0)
+    (property "Value" "LVS303015-2R2M" (at 214.63 68.58 0)
       (effects (font (size 1.27 1.27)))
     )
-    (property "Footprint" "MAS_Package_std:Power_inductor_SMD_0530" (at 214.63 84.455 0)
+    (property "Footprint" "Inductor_SMD:L_Wuerth_MAPI-3015" (at 214.63 84.455 0)
       (effects (font (size 1.27 1.27) italic) hide)
     )
-    (property "Datasheet" "https://datasheet.lcsc.com/lcsc/1811151233_Sunltech-Tech-SLO0530H6R8MTT_C325965.pdf" (at 214.63 86.36 0)
+    (property "Datasheet" "https://datasheet.lcsc.com/lcsc/1811021412_Chilisin-Elec-LVS303015-2R2M-N_C285837.pdf" (at 214.63 86.36 0)
       (effects (font (size 1.27 1.27) italic) hide)
     )
-    (property "lcsc" "C325962" (at 214.63 71.12 0)
+    (property "lcsc" "C285837" (at 214.63 71.12 0)
       (effects (font (size 1.27 1.27)) hide)
     )
@@
     )
   )
-  (symbol (lib_id "pspice:INDUCTOR") (at 314.96 71.12 0) (unit 1)
-    (in_bom yes) (on_board yes) (dnp no)
-    (property "Reference" "L6" (at 314.96 66.04 0)
-      (effects (font (size 1.27 1.27)))
-    )
-    (property "Value" "SLO0530H2R2MTT" (at 314.96 68.58 0)
-      (effects (font (size 1.27 1.27)))
-    )
-    (property "Footprint" "MAS_Package_std:Power_inductor_SMD_0530" (at 314.96 84.455 0)
-      (effects (font (size 1.27 1.27) italic) hide)
-    )
-    (property "Datasheet" "https://datasheet.lcsc.com/lcsc/1811151233_Sunltech-Tech-SLO0530H6R8MTT_C325965.pdf" (at 314.96 86.36 0)
-      (effects (font (size 1.27 1.27) italic) hide)
-    )
-    (property "lcsc" "C325962" (at 314.96 71.12 0)
-      (effects (font (size 1.27 1.27)) hide)
-    )
-    (pin "1")
-    (pin "2")
-    (instances
-      (project "main"
-        (path "/c6e5d5ba-43a3-4ff8-a766-3efdb024d1f4/f32ecbe8-471f-4b0d-831c-9a3a555bc765"
-          (reference "L6") (unit 1)
-        )
-      )
-    )
-  )
   (symbol (lib_id "Device:C_Small") (at 251.46 -29.21 0) (unit 1)
     (in_bom yes) (on_board yes) (dnp no)
@@
     )
   )
-  (symbol (lib_id "pspice:INDUCTOR") (at 214.63 107.95 0) (unit 1)
-    (in_bom yes) (on_board yes) (dnp no)
-    (property "Reference" "L5" (at 214.63 102.87 0)
-      (effects (font (size 1.27 1.27)))
-    )
-    (property "Value" "SLO0530H2R2MTT" (at 214.63 105.41 0)
-      (effects (font (size 1.27 1.27)))
-    )
-    (property "Footprint" "MAS_Package_std:Power_inductor_SMD_0530" (at 214.63 121.285 0)
-      (effects (font (size 1.27 1.27) italic) hide)
-    )
-    (property "Datasheet" "https://datasheet.lcsc.com/lcsc/1811151233_Sunltech-Tech-SLO0530H6R8MTT_C325965.pdf" (at 214.63 123.19 0)
-      (effects (font (size 1.27 1.27) italic) hide)
-    )
-    (property "lcsc" "C325962" (at 214.63 107.95 0)
-      (effects (font (size 1.27 1.27)) hide)
-    )
-    (pin "1")
-    (pin "2")
-    (instances
-      (project "main"
-        (path "/c6e5d5ba-43a3-4ff8-a766-3efdb024d1f4/f32ecbe8-471f-4b0d-831c-9a3a555bc765"
-          (reference "L5") (unit 1)
-        )
-      )
-    )
-  )
   (symbol (lib_id "Device:C_Small") (at 265.43 77.47 0) (unit 1)
     (in_bom yes) (on_board yes) (dnp no)
@@
     )
   )
-  (symbol (lib_id "pspice:INDUCTOR") (at 314.96 107.95 0) (unit 1)
-    (in_bom yes) (on_board yes) (dnp no)
-    (property "Reference" "L7" (at 314.96 102.87 0)
-      (effects (font (size 1.27 1.27)))
-    )
-    (property "Value" "SLO0530H2R2MTT" (at 314.96 105.41 0)
-      (effects (font (size 1.27 1.27)))
-    )
-    (property "Footprint" "MAS_Package_std:Power_inductor_SMD_0530" (at 314.96 121.285 0)
-      (effects (font (size 1.27 1.27) italic) hide)
-    )
-    (property "Datasheet" "https://datasheet.lcsc.com/lcsc/1811151233_Sunltech-Tech-SLO0530H6R8MTT_C325965.pdf" (at 314.96 123.19 0)
-      (effects (font (size 1.27 1.27) italic) hide)
-    )
-    (property "lcsc" "C325962" (at 314.96 107.95 0)
-      (effects (font (size 1.27 1.27)) hide)
-    )
-    (pin "1")
-    (pin "2")
-    (instances
-      (project "main"
-        (path "/c6e5d5ba-43a3-4ff8-a766-3efdb024d1f4/f32ecbe8-471f-4b0d-831c-9a3a555bc765"
-          (reference "L7") (unit 1)
-        )
-      )
-    )
-  )
   (symbol (lib_id "Device:C_Small") (at 165.1 77.47 0) (unit 1)
     (in_bom yes) (on_board yes) (dnp no)
@@
     )
   )
+  (symbol (lib_id "pspice:INDUCTOR") (at 314.96 71.12 0) (unit 1)
+    (in_bom yes) (on_board yes) (dnp no)
+    (property "Reference" "L6" (at 314.96 66.04 0)
+      (effects (font (size 1.27 1.27)))
+    )
+    (property "Value" "LVS303015-2R2M" (at 314.96 68.58 0)
+      (effects (font (size 1.27 1.27)))
+    )
+    (property "Footprint" "Inductor_SMD:L_Wuerth_MAPI-3015" (at 314.96 84.455 0)
+      (effects (font (size 1.27 1.27) italic) hide)
+    )
+    (property "Datasheet" "https://datasheet.lcsc.com/lcsc/1811021412_Chilisin-Elec-LVS303015-2R2M-N_C285837.pdf" (at 314.96 86.36 0)
+      (effects (font (size 1.27 1.27) italic) hide)
+    )
+    (property "lcsc" "C285837" (at 314.96 71.12 0)
+      (effects (font (size 1.27 1.27)) hide)
+    )
+    (pin "1")
+    (pin "2")
+    (instances
+      (project "main"
+        (path "/c6e5d5ba-43a3-4ff8-a766-3efdb024d1f4/f32ecbe8-471f-4b0d-831c-9a3a555bc765"
+          (reference "L6") (unit 1)
+        )
+      )
+    )
+  )
+  (symbol (lib_id "pspice:INDUCTOR") (at 214.63 107.95 0) (unit 1)
+    (in_bom yes) (on_board yes) (dnp no)
+    (property "Reference" "L5" (at 214.63 102.87 0)
+      (effects (font (size 1.27 1.27)))
+    )
+    (property "Value" "LVS303015-2R2M" (at 214.63 105.41 0)
+      (effects (font (size 1.27 1.27)))
+    )
+    (property "Footprint" "Inductor_SMD:L_Wuerth_MAPI-3015" (at 214.63 121.285 0)
+      (effects (font (size 1.27 1.27) italic) hide)
+    )
+    (property "Datasheet" "https://datasheet.lcsc.com/lcsc/1811021412_Chilisin-Elec-LVS303015-2R2M-N_C285837.pdf" (at 214.63 123.19 0)
+      (effects (font (size 1.27 1.27) italic) hide)
+    )
+    (property "lcsc" "C285837" (at 214.63 107.95 0)
+      (effects (font (size 1.27 1.27)) hide)
+    )
+    (pin "1")
+    (pin "2")
+    (instances
+      (project "main"
+        (path "/c6e5d5ba-43a3-4ff8-a766-3efdb024d1f4/f32ecbe8-471f-4b0d-831c-9a3a555bc765"
+          (reference "L5") (unit 1)
+        )
+      )
+    )
+  )
   (symbol (lib_id "Device:C_Small") (at 271.78 -57.15 0) (unit 1)
     (in_bom yes) (on_board yes) (dnp no)
@@
         )
       )
+    )
+  )
+  (symbol (lib_id "pspice:INDUCTOR") (at 314.96 107.95 0) (unit 1)
+    (in_bom yes) (on_board yes) (dnp no)
+    (property "Reference" "L7" (at 314.96 102.87 0)
+      (effects (font (size 1.27 1.27)))
+    )
+    (property "Value" "LVS303015-2R2M" (at 314.96 105.41 0)
+      (effects (font (size 1.27 1.27)))
+    )
+    (property "Footprint" "Inductor_SMD:L_Wuerth_MAPI-3015" (at 314.96 121.285 0)
+      (effects (font (size 1.27 1.27) italic) hide)
+    )
+    (property "Datasheet" "https://datasheet.lcsc.com/lcsc/1811021412_Chilisin-Elec-LVS303015-2R2M-N_C285837.pdf" (at 314.96 123.19 0)
+      (effects (font (size 1.27 1.27) italic) hide)
+    )
+    (property "lcsc" "C285837" (at 314.96 107.95 0)
+      (effects (font (size 1.27 1.27)) hide)
+    )
+    (pin "1")
+    (pin "2")
+    (instances
+      (project "main"
+        (path "/c6e5d5ba-43a3-4ff8-a766-3efdb024d1f4/f32ecbe8-471f-4b0d-831c-9a3a555bc765"
+          (reference "L7") (unit 1)
+        )
+      )

Commit message: update pcb
Parts:
- removed R17: 100k, Resistor_SMD:R_0402_1005Metric, symbol Device:R_Small
- added D3: MBR0540, Diode_SMD:D_SOD-123, symbol Diode:MBR0540
- added R125: 10k, Resistor_SMD:R_0402_1005Metric, symbol Device:R_Small
Connections:
- net +3V3: now also R125.1
- net +5V: now also C34.1
- net at C9.1, R12.1, SW2.2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: now also D3.1 (K)
- net at C28.1, C52.1, C52.1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: no longer C34.1
- new net WPS: D3.2 (A), R125.2
- no-connect marks 0 -> 1
Other:
- note added: "!!!!!!!!!!!!"
- moved on the sheet: C34, JP2
