File: hardware/main.kicad_sch (KiCad schematic)
At the start: 13 parts, among them J4 98424-G52-04ALF

Commit message: circuits are combined
Parts:
- added C1, C103, C115, C119, C120, C123, C124, C125, C127, C14, C15, C17, C30, C31, C36, C37, C4, C47, C48, C7, C75, C76, C81, C82, C85: 10u, Capacitor_SMD:C_0603_1608Metric, symbol Device:C_Small
- added C10, C100, C101, C102, C104, C106, C109, C11, C110, C111, C112, C113, C114, C117, C118, C12, C121, C122, C13, C159, C16, C160, C161, C162, C164, C165, C166, C167, C168, C169, C170, C171, C172, C173, C178, C18, C183, C184, C185, C19, C194, C196, C197, C2, C20, C21, C22, C26, C27, C28, C29, C3, C38, C39, C42, C43, C44, C49, C50, C53, C54, C57, C58, C59, C60, C61, C62, C63, C64, C65, C66, C67, C68, C69, C70, C71, C72, C73, C74, C77, C78, C79, C8, C80, C83, C84, C86, C87, C88, C89, C9, C90, C91, C92, C93, C94, C95, C96, C97, C98, C99: 100n, Capacitor_SMD:C_0402_1005Metric, symbol Device:C_Small
- added C105, C107, C108: 1n, Capacitor_SMD:C_0805_2012Metric, symbol Device:C_Small
- added C116, C128, C129, C130, C131, C132, C133, C134, C135, C136, C137, C138, C139, C23, C32, C33, C45, C46, C5, C52, C6: 4.7u, Capacitor_SMD:C_0603_1608Metric, symbol Device:C_Small
- added C140, C141, C55, C56: 470n, Capacitor_SMD:C_0402_1005Metric, symbol Device:C_Small
- added C174, C175: 18p, Capacitor_SMD:C_0402_1005Metric, symbol Device:C_Small
- added C186, C189, C191: 22u, Capacitor_SMD:C_0805_2012Metric, symbol Device:C_Small
- added C190, C192: 10u, Capacitor_SMD:C_0805_2012Metric, symbol Device:C_Small
- added C24, C25: 4.7p, Capacitor_SMD:C_0402_1005Metric, symbol Device:C_Small
- added C34: 100u, Capacitor_Tantalum_SMD:CP_EIA-7343-31_Kemet-D, symbol Device:C_Polarized_Small
- added C35: 100uF, Capacitor_Tantalum_SMD:CP_EIA-3528-21_Kemet-B, symbol main-rescue:CP_Small-Device
- added C40, C41, C51, C52: 22p, Capacitor_SMD:C_0402_1005Metric, symbol Device:C_Small
- added D1 (x2): LEDY, Diode_SMD:D_0603_1608Metric, symbol Device:LED_Small
- added D3 (x2): MBR0540, Diode_SMD:D_SOD-123, symbol Diode:MBR0540
- added J1, J2, J3: DS1128-09-S8B8X, MAS_Package_std:RJ45_DS1128-09-S8B8X, symbol MAS_Connectors:DS1128-09-S8B8X
- added J10: AS0BC21-S30BM-7H, MAS_Package_std:Bus_M.2_Socket_M, symbol Connector:Bus_M.2_Socket_M
- added J5: miniPCI-E_52P_5.2, MAS_Package_std:BUS_PCI_Express_Mini_Dual, symbol Connector:Bus_PCI_Express_Mini
- added J6, J7: IDC-08M, Connector_PinHeader_1.27mm:PinHeader_2x04_P1.27mm_Vertical, symbol Connector_Generic:Conn_02x04_Counter_Clockwise
- added J8: USB_C_Receptacle, Connector_USB:USB_C_Receptacle_HRO_TYPE-C-31-M-12, symbol Connector:USB_C_Receptacle
- added J9: TYPE-C-31-M-12, MAS_Package_std:USB_C_Receptacle_HRO_TYPE-C-31-M-12, symbol Connector:USB_C_Receptacle_USB2.0
- added JP1, JP2, JP3, JP4, JP5, JP6, JP7: JP, MAS_Package_nostd:SolderJumper_Open_Pad0.5x0.8mm, symbol Jumper:Jumper_2_Open
- added L1, L26: SLO0530H2R2MTT, MAS_Package_std:Power_inductor_SMD_0530, symbol pspice:INDUCTOR
- added L2: SLO0530H1R0MTT, MAS_Package_std:Power_inductor_SMD_0530, symbol pspice:INDUCTOR
- added L3, L8: CBM160808U121T, Inductor_SMD:L_0603_1608Metric, symbol pspice:INDUCTOR
- added L4, L5, L6, L7: LVS303015-2R2M, Inductor_SMD:L_Wuerth_MAPI-3015, symbol pspice:INDUCTOR
- added Q1, Q2: SSM6J501NU, MAS_Package_std:U-MOSVI, symbol MAS_Transistors:SSM6J501NU
- added Q3: FDV301N, Package_TO_SOT_SMD:SOT-23, symbol MAS_Transistors:FDV301N
- added R1, R10, R11, R116 (x2), R12, R13, R14, R15, R16, R20, R44, R45, R6, R7, R90: 1k, Resistor_SMD:R_0402_1005Metric, symbol Device:R_Small
- added R100, R103, R47: 24k, Resistor_SMD:R_0402_1005Metric, symbol Device:R_Small
- added R101, R102: 22k, Resistor_SMD:R_0402_1005Metric, symbol Device:R_Small
- added R104, R105, R106, R107, R108, R113, R114, R161, R165, R168, R169, R170, R171, R3 (x4), R69, R70, R98, R99: 0R, Resistor_SMD:R_0402_1005Metric, symbol Device:R_Small
- added R109, R110, R111, R112, R68, R71: 51R, Resistor_SMD:R_0402_1005Metric, symbol Device:R_Small
- added R115, R125, R18, R4, R9: 10k, Resistor_SMD:R_0402_1005Metric, symbol Device:R_Small
- added R117: 0.01R, Resistor_SMD:R_1206_3216Metric, symbol Device:R_Small
- added R118: 82k, Resistor_SMD:R_0402_1005Metric, symbol Device:R_Small
- added R119, R128, R26, R27, R28, R30, R32, R33, R36, R37, R39: 100k, Resistor_SMD:R_0402_1005Metric, symbol Device:R_Small
- added R120: 100k (NTC), Resistor_SMD:R_0805_2012Metric, symbol MAS_Resistors:Thermistor_NTC
- added R121, R130, R131, R134, R136, R137, R139, R141, R143, R146, R147, R150, R152, R154, R156, R157, R160, R162, R172, R40, R41, R46, R49, R8: ~, Resistor_SMD:R_0402_1005Metric, symbol Device:R_Small
- added R122, R123, R129, R132, R133, R135, R138, R140, R142, R144, R145, R148, R149, R151, R153, R155, R158, R159, R163, R166, R167, R42, R43, R48, R87 (x2): 4.7k, Resistor_SMD:R_0402_1005Metric, symbol Device:R_Small
- added R124, R5: 470R, Resistor_SMD:R_0402_1005Metric, symbol Device:R_Small
- added R164: 910k, Resistor_SMD:R_0402_1005Metric, symbol Device:R_Small
- added R19: 1.1k, Resistor_SMD:R_0402_1005Metric, symbol Device:R_Small
- added R2, R35: 240R, Resistor_SMD:R_0402_1005Metric, symbol Device:R_Small
- added R21: 330k, Resistor_SMD:R_0402_1005Metric, symbol Device:R_Small
- added R22: 51k, Resistor_SMD:R_0402_1005Metric, symbol Device:R_Small
- added R23: 2k, Resistor_SMD:R_0402_1005Metric, symbol Device:R_Small
- added R24, R25: 68k, Resistor_SMD:R_0402_1005Metric, symbol Device:R_Small
- added R29: 120k, Resistor_SMD:R_0402_1005Metric, symbol Device:R_Small
- added R31, R38: 150k, Resistor_SMD:R_0402_1005Metric, symbol Device:R_Small
- added R34: 100R, Resistor_SMD:R_0402_1005Metric, symbol Device:R_Small
- added R50, R51, R52, R53, R54, R55, R56, R57, R58, R59, R60, R61: 75R, Resistor_SMD:R_0402_1005Metric, symbol Device:R_Small
- added R62, R63, R64, R65, R66, R67: 330R, Resistor_SMD:R_0402_1005Metric, symbol Device:R_Small
- added R91, R92, R93, R94, R95, R96, R97: 22R, Resistor_SMD:R_0402_1005Metric, symbol Device:R_Small
- added RN1: 4D03WGJ0102T5E, Resistor_SMD:R_Array_Convex_4x0603, symbol Device:R_Pack04
- added SW1, SW2, SW4: TS-1187A-B-A-B, Button_Switch_SMD:SW_SPST_TL3342, symbol Switch:SW_Push
- added TP1, TP10, TP11, TP12, TP13, TP14, TP15, TP16, TP17, TP18, TP19, TP2, TP20, TP21, TP22, TP23, TP24, TP25, TP26, TP27, TP28, TP29, TP3, TP30, TP31, TP32, TP33, TP34, TP4, TP5, TP6, TP7, TP8, TP9: TP, MAS_Package_std:TestPoint_Pad_D1mm, symbol Connector:TestPoint
- added TR1, TR2, TR3: H2450G, MAS_Package_nostd:Transformer_Ethernet_E-NETTR_24, symbol MAS_Transformers:H2450G
- added U1: SN74LVC1G175, Package_TO_SOT_SMD:SOT-23-6, symbol MAS_IC_Logic:SN74LVC1G175
- added U10: W25Q256FVEIG, MAS_Package_std:WSON-8-1EP_8x6mm_P1.27mm_EP3.4x4mm, symbol MAS_IC_Memory:W25Qx
- added U12, U13, U14: TPD2EUSB30, Package_TO_SOT_SMD:Texas_DRT-3, symbol Power_Protection:TPD2EUSB30
- added U15: IP5328P, Package_DFN_QFN:QFN-40-1EP_6x6mm_P0.5mm_EP4.6x4.6mm, symbol MAS_IC_PowerSupply:IP5328P
- added U16: N096-2864KSWEG01-H30, MAS_Package_nostd:SSD1306-oled-0.96, symbol MAS_Module:SSD1306-OLED-0.96
- added U2: MT7621A, MAS_Package_std:TFBGA-387_11.7x13.6mm_P0.65mm, symbol MAS_IC_MCU:MT7621A
- added U3, U4: TPS63020, Package_DFN_QFN:DFN-14-1EP_3x4mm_P0.5mm_EP1.7x3.3mm, symbol MAS_IC_PowerSupply:TPS6302x
- added U5, U6, U7, U8: MT3420B, Package_TO_SOT_SMD:SOT-23-6, symbol MAS_IC_PowerSupply:MT3420
- added U9: NT5CB64M16FP-DH (!), Package_BGA:BGA-96_9.0x13.0mm_Layout2x3x16_P0.8mm, symbol Memory_RAM:AS4C256M16D3
- added Y1: X322540MPB4SI, MAS_Package_std:Oscillator_SMD_SMD3225-4P, symbol Device:Crystal_GND24
Connections:
- net +BATT: now also C119.1, C123.2, C124.1, C189.2, C190.1, C191.2, C192.1, C2.1, L26.2, Q2.4 (S1), Q2.7 (S1), R12.2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
- net -BATT: now also C1.2, C10.2, C100.1, C101.1, C103.2, C11.2, C115.2, C116.2, C117.2, C118.2, C119.2, C12.2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
- new net: J5.7 (~{CLKREQ}), TP15.1
- new net: C121.1, C76.1, J5.47 (Reserved), J5.49 (Reserved), R3.1
- new net: C107.2, R54.1, R55.1, R56.1, R57.1
- new net: R118.2, R120.1, U15.10 (NTC)
- new net: C185.2, L26.1, U15.14 (LX), U15.15 (LX), U15.16 (LX), U15.17 (LX), U15.18 (LX)
- new net: C185.1, U15.19 (BST)
- new net: D1.2 (A), U15.20 (LIGHT)
- new net: R119.1, U15.21 (RSET)
- new net: C102.2, C104.2, C106.2, C109.2, C110.2, C134.2, C135.2, C136.2, C87.2, C93.2
- new net: R6.1, U3.13 (PS/SYNC)
- new net: C20.1, R1.2, R6.2, U3.1 (VINA)
- new net: TP20.1, U2.H3 (RXD3)
- new net: C40.2, R28.1, R29.2, U5.6 (FB)
- new net: C108.2, R58.1, R59.1, R60.1, R61.1
- new net: R59.2, TR3.16 (MX3-)
- new net: R58.2, TR3.15 (CT)
- new net: C29.1, C32.1, C35.1, C45.1, JP3.2 (B), R21.2, R25.1, U4.4 (VOUT), U4.5 (VOUT)
- new net: C94.2, TR3.10 (CT)
- new net: R60.2, TR3.21 (CT)
- new net: R61.2, TR3.22 (MX1-)
- new net: C97.2, TR3.3 (TD1-)
- new net: C96.2, TR3.4 (CT)
- new net: C95.2, TR3.9 (TD3-)
- new net: C79.1, C80.1, R46.1, U2.M7 (DVDD_GE1_IO), U2.M8 (DVDD_GE1_IO)
- new net: C105.2, R50.1, R51.1, R52.1, R53.1
- new net: R51.2, TR1.16 (MX3-)
- new net: C9.1, D3.1 (K), R12.1, SW2.2, U1.1 (CLK)
- new net: Q2.3 (G1), Q3.3 (D), R4.2, U1.3 (D)
- new net: R5.1, U1.4 (Q)
- new net: C51.2, R36.1, R37.2, U7.6 (FB)
- new net: C125.1, C51.1, C53.1, JP6.2 (B), L6.2, R36.2
- new net: C41.2, R30.1, R31.2, U6.6 (FB)
- new net: C30.1, C41.1, C44.1, JP5.2 (B), L5.2, R30.2
- new net: TP3.1, U2.F1 (~{ND_RB})
- new net: R54.2, TR2.15 (CT)
- new net: TP12.1, U2.T13 (SCL)
- new net: C28.1, C33.1, C6.1, JP2.2 (B), R18.2, R24.1, U3.4 (VOUT), U3.5 (VOUT)
- new net: C141.2, C178.2, R113.2, U2.J1 (AVDD12_SSUSB)
- new net: C138.1, U16.28 (VDisplay)
- new net: R170.2, U16.12 (BS2)
- new net: TP19.1, U2.H1 (TXD3)
- new net: R33.1, U8.1 (EN)
- new net: R50.2, TR1.15 (CT)
- new net: C90.2, TR1.9 (TD3-)
- new net: C78.1, R44.1, R45.2, U2.M6 (DVDD_GE1_VREF)
- new net: C83.1, C84.1, C86.1, C88.1, L3.2, U2.U10 (AVDD33_LD_P4), U2.U5 (AVDD33_LD_P0), U2.U6 (AVDD33_LD_P1), U2.U7 (AVDD33_LD_P2), U2.U8 (AVDD33_PLL_1), U2.U9 (AVDD33_LD_P3)
- new net: L7.1, U8.3 (LX)
- new net: C52.2, R38.1, R39.2, U8.6 (FB)
- new net: C197.1, R162.1, R163.1, U16.14 (Reset)
- new net: J7.7 (Pin_7), R97.1, RN1.2 (R2.1)
- new net: R97.2, U2.G17 (JTDO)
- new net: R16.1, U4.13 (PS/SYNC)
- new net: C21.1, R16.2, R7.2, U4.1 (VINA)
- new net: C164.1, U2.L18 (PCIE_TXP1)
- new net: TP6.1, U2.F2 (ND_D0)
- new net: J3.10, R64.2
- new net: J1.12, R65.2
- new net: J8.A5 (CC1), R101.1
- new net: C175.1, U2.P18 (XPTL_XO), Y1.1
- new net: C174.1, U2.P17 (XPTL_XI), Y1.3
- new net: C24.2, R18.1, R19.1, U3.3 (FB)
- new net: J3.12, R67.2
- new net: C160.1, J8.A2 (TX1+), J8.B2 (TX2+)
- new net: C159.2, J8.A3 (TX1-), J8.B3 (TX2-)
- new net: J8.B5 (CC2), R102.1
- new net: TP11.1, U2.V5 (ESW_TANA)
- new net: L1.1, U3.8 (L1), U3.9 (L1)
- new net: L1.2, U3.6 (L2), U3.7 (L2)
- new net: R69.2, U2.M13 (PCIE_CKP2)
- new net: R32.1, U7.1 (EN)
- new net: R169.2, U16.11 (BS1)
- new net: C112.1, U2.N17 (PCIE_TXN2)
- new net: J2.12, R66.2
- new net: J5.51 (Reserved), TP18.1
- new net: J10.10 (DAS/~{DSS}/~{LED1}), TP30.1
- new net: R1.1, U3.12 (EN)
- new net: C89.2, TR1.10 (CT)
- new net: R52.2, TR1.21 (CT)
- new net: R53.2, TR1.22 (MX1-)
- new net: C92.2, TR1.3 (TD1-)
- new net: C91.2, TR1.4 (CT)
- new net: TP1.1, U2.E18 (TN_MEMPLL)
- new net: C137.1, U16.27 (VCOMH)
- new net: R105.2, U2.K14 (PCIE_CKN1)
- new net: J2.10, R63.2
- new net: TP4.1, U2.G3 (ND_CLE)
- new net: C140.1, C168.1, R108.2, U2.K4 (AVDD33_SSUSB), U2.K5 (AVDD33_USB), U2.K6 (AVDD33_XDRV)
- new net: L6.1, U7.3 (LX)
- new net: D1.1 (K), R116.2
- new net: D1.2 (A), J5.44 (~{LED_WLAN})
- new net: R168.2, U16.10 (BS0)
- new net: TP21.1, U2.H5 (CTS3_N)
- new net: R107.2, U2.H13 (PCIE_CKN0)
- new net: R7.1, U4.12 (EN)
- new net: L2.1, U4.8 (L1), U4.9 (L1)
- new net: L2.2, U4.6 (L2), U4.7 (L2)
- new net: C98.2, TR2.10 (CT)
- new net: R55.2, TR2.16 (MX3-)
- new net: R56.2, TR2.21 (CT)
- new net: R57.2, TR2.22 (MX1-)
- new net: C101.2, TR2.3 (TD1-)
- new net: C100.2, TR2.4 (CT)
- new net: C99.2, TR2.9 (TD3-)
- new net: TP7.1, U2.E3 (ND_D1)
- new net: Q3.1 (G), R5.2
- new net: R116.1, SW1.1
- new net: J10.50 (~{PERST}), R3.2, R87.1
- new net: L5.1, U6.3 (LX)
- new net: C127.1, C52.1, C54.1, JP7.2 (B), L7.2, R38.2
- new net: R3.1, U2.C3 (DVDD_VREF)
- new net: C25.2, R21.1, R22.1, U4.3 (FB)
- new net: R98.1, U2.P13 (I2C_SCLK)
- new net: C24.1, R24.2
- new net: C40.1, C43.1, C7.1, JP4.2 (B), L4.2, R28.2
- new net: R103.1, U2.L2 (SSUSB_VRT)
- new net: R164.2, U16.26 (IREF)
- new net: C169.2, C56.2, R114.2, U2.J18 (AVDD12_PE)
- new net: R26.1, U5.1 (EN)
- new net: L4.1, U5.3 (LX)
- new net: R100.1, U2.L16 (CBG_VRT)
- new net: R171.2, U16.13 (C/S)
- new net: R165.2, R172.2, U16.15 (D/C)
- new net: C129.2, U16.2 (C2P)
- new net: C129.1, U16.3 (C2N)
- new net: C130.2, U16.4 (C1P)
- new net: C130.1, U16.5 (C1N)
- new net: R8.1, R9.1, U2.F4 (ND_WP)
- new net: C111.1, U2.N16 (PCIE_TXP2)
- new net: J5.20 (~{W_DISABLE}), TP16.1
- new net: R92.2, U2.R13 (RXD1)
- new net: J5.45 (Reserved), TP17.1
- new net: TP23.1, U2.L10 (CBG_AVOUTP)
- new net: J10.52 (~{CLKREQ}), TP26.1
- new net: C167.1, U2.H17 (PCIE_TXN0)
- new net: TP9.1, U2.E4 (ND_D3)
- new net: C25.1, R25.2
- new net: J7.1 (Pin_1), RN1.4 (R4.1), U2.F16 (JTCLK)
- new net: J7.5 (Pin_5), R90.2, U2.F17 (JTRST_N)
- new net: J7.6 (Pin_6), RN1.1 (R1.1), U2.G16 (JTDI)
- new net: J7.8 (Pin_8), RN1.3 (R3.1), U2.G18 (JTMS)
- new net: J1.10, R62.2
- new net: R104.2, U2.K13 (PCIE_CKP1)
- new net: J5.22 (~{PERST}), R3.2, R87.1
- new net: R106.2, U2.H14 (PCIE_CKP0)
- new net: C166.1, U2.H16 (PCIE_TXP0)
- new net: R94.2, U2.H4 (RXD2)
- new net: C173.1, U2.J16 (PCIE_RXN0)
- new net: C172.1, U2.J17 (PCIE_RXP0)
- new net: R95.2, U2.J5 (CTS2_N)
- new net: C171.1, U2.K16 (PCIE_RXN1)
- new net: C170.1, U2.K17 (PCIE_RXP1)
- new net: TP24.1, U2.L11 (CBG_AVOUTN)
- new net: C165.1, U2.L17 (PCIE_TXN1)
- new net: R70.2, U2.M14 (PCIE_CKN2)
- new net: C113.1, U2.M17 (PCIE_RXP2)
- new net: C114.1, U2.M18 (PCIE_RXN2)
- new net: R99.2, U2.P14 (I2C_SD)
- new net: R2.2, U2.B1 (REXTDN)
- new net: TP2.1, U2.E17 (TP_MEMPLL)
- new net: TP8.1, U2.E2 (ND_D2)
- new net: TP5.1, U2.G5 (ND_ALE)
- new net: TP14.1, U2.V7 (ESW_XI)
- new net: R47.1, U2.W5 (ESW_REXT)
- new net: R22.2, R23.1
- new net: R35.2, U9.L8 (ZQ)
- new net: D1.1 (K), R124.2
- new net: R48.2, R49.2, TP10.1, U2.T12 (A_POR_BPS)
- new net: J10.54 (~{PEWAKE}), TP27.1
- new net: J5.1 (~{WAKE}), TP25.1
- new net: TP13.1, U2.V8 (ESW_XO)
- new net: R27.1, U6.1 (EN)
- new net +1V0: C102.1, C104.1, C106.1, C109.1, C110.1, C115.1, C12.1, C134.1, C135.1, C136.1, C8.1, C87.1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
- new net +1V1: C10.1, C13.1, C22.1, C26.1, C27.1, C42.1, C85.1, JP4.1 (A), U2.F7 (DVDDK), U2.F8 (DVDDK), U2.G12 (DVDDK), U2.G8 (DVDDK)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
- new net +1V2: JP6.1 (A), R113.1, R114.1
- new net +1V5: C103.1, C11.1, C116.1, C118.1, C16.1, C3.1, C46.1, C57.1, C58.1, C60.1, C61.1, C62.1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
- new net +3V3: C117.1, C122.1, C128.1, C14.1, C162.1, C31.1, C36.1, C37.1, C38.1, C39.1, C47.1, C48.1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
- new net +5V: C139.1, C161.1, C34.1, J8.A4 (VBUS), J8.A9 (VBUS), J8.B4 (VBUS), J8.B9 (VBUS), JP2.1 (A), R101.2, R102.2, R3.2
- new net 3V3O: C131.1, C132.2, C133.2, C196.1, R161.1, R163.2, R165.1, R166.2, R167.2, R169.1, U16.6 (VPump), U16.9 (VLogic)
- new net CC1: J9.A5 (CC1), U15.3 (CC2)
- new net CC2: J9.B5 (CC2), U15.2 (CC1)
- new net CTS2: J6.6 (Pin_6), R95.1
- new net D2DB_PORST_N: C194.1, D3.2 (A), J7.2 (Pin_2), R128.2, SW4.1, U2.R12 (PORST_N), U4.14 (PG)
- new net DDR3RSTB: U2.D11 (DDR3RSTB), U9.T2 (~{RESET})
- new net DDRVREF: C73.1, R15.1, R20.2, R3.2
- new net DDR_VREF1: C66.1, R13.1, R14.2, U9.M8 (VREFCA)
- new net DDR_VREF2: C59.1, R10.1, R11.2, U9.H1 (VREFDQ)
- new net DMC: J9.A7 (D-), J9.B7 (D-), U15.4 (DMC)
- new net DPC: J9.A6 (D+), J9.B6 (D+), U15.5 (DPC)
- new net EN_DC: U2.V16 (GE2_TXEN)
- new net ESW_TXVN_A_P2: TR1.11 (TD4+), U2.AA3 (ESW_TXVN_A_P2)
- new net ESW_TXVN_A_P3: TR2.11 (TD4+), U2.Y8 (ESW_TXVN_A_P3)
- new net ESW_TXVN_A_P4: TR3.11 (TD4+), U2.Y11 (ESW_TXVN_A_P4)
- new net ESW_TXVN_B_P2: TR1.7 (CT), U2.W3 (ESW_TXVN_B_P2)
- new net ESW_TXVN_B_P3: TR2.7 (CT), U2.Y9 (ESW_TXVN_B_P3)
- new net ESW_TXVN_B_P4: TR3.7 (CT), U2.W12 (ESW_TXVN_B_P4)
- new net ESW_TXVN_C_P2: TR1.5 (TD2+), U2.Y6 (ESW_TXVN_C_P2)
- new net ESW_TXVN_C_P3: TR2.5 (TD2+), U2.AA10 (ESW_TXVN_C_P3)
- new net ESW_TXVN_C_P4: TR3.5 (TD2+), U2.Y13 (ESW_TXVN_C_P4)
- new net ESW_TXVN_D_P2: TR1.1 (CT), U2.Y7 (ESW_TXVN_D_P2)
- new net ESW_TXVN_D_P3: TR2.1 (CT), U2.W10 (ESW_TXVN_D_P3)
- new net ESW_TXVN_D_P4: TR3.1 (CT), U2.Y14 (ESW_TXVP_D_P4)
- new net ESW_TXVP_A_P2: TR1.12 (TD4-), U2.AA2 (ESW_TXVP_A_P2)
- new net ESW_TXVP_A_P3: TR2.12 (TD4-), U2.W8 (ESW_TXVP_A_P3)
- new net ESW_TXVP_A_P4: TR3.12 (TD4-), U2.AA11 (ESW_TXVP_A_P4)
- new net ESW_TXVP_B_P2: TR1.8 (TD3+), U2.Y3 (ESW_TXVP_B_P2)
- new net ESW_TXVP_B_P3: TR2.8 (TD3+), U2.W9 (ESW_TXVP_B_P3)
- new net ESW_TXVP_B_P4: TR3.8 (TD3+), U2.Y12 (ESW_TXVP_B_P4)
- new net ESW_TXVP_C_P2: TR1.6 (TD2-), U2.W6 (ESW_TXVP_C_P2)
- new net ESW_TXVP_C_P3: TR2.6 (TD2-), U2.Y10 (ESW_TXVP_C_P3)
- new net ESW_TXVP_C_P4: TR3.6 (TD2-), U2.AA13 (ESW_TXVP_C_P4)
- new net ESW_TXVP_D_P2: TR1.2 (TD1+), U2.W7 (ESW_TXVP_D_P2)
- new net ESW_TXVP_D_P3: TR2.2 (TD1+), U2.V10 (ESW_TXVP_D_P3)
- new net ESW_TXVP_D_P4: TR3.2 (TD1+), U2.W14 (ESW_TXVN_D_P4)
- new net G2-: J1.9, R153.2, R154.2, U2.W15 (ESW_P2_LED_0)
- new net G3-: J2.9, R157.2, R158.2, U2.AA15 (ESW_P3_LED_0)
- new net G4-: J3.9, R159.2, R160.2, U2.Y15 (ESW_P4_LED_0)
- new net GNDREF: C105.1, C107.1, C108.1, J1.13, J1.14, J2.13, J2.14, J3.13, J3.14
- new net GPIO0: R147.2, R148.2, U2.P12 (GPIO0)
- new net INT: R121.1, TP34.1, U15.13 (L3), U2.V18 (GE2_TXCLK)
- new net KEY: R116.2, U15.26 (KEY)
- new net MDC: R135.2, R136.2, U2.T15 (MDC)
- new net ND_CS_N: R133.2, R134.2, R41.1, U10.1 (CS), U2.G2 (~{ND_CS})
- new net ND_D4: R40.2, U10.2 (DO(IO1)), U2.D1 (ND_D4)
- new net ND_D5: U10.5 (DI(IO0)), U2.D2 (ND_D5)
- new net ND_D6: R43.1, U10.3 (WP(IO2)), U2.C1 (ND_D6)
- new net ND_D7: R42.1, U10.7 (HOLD(IO3)), U2.D3 (ND_D7)
- new net ND_RE_N: R129.2, R130.2, U10.6 (CLK), U2.F3 (~{ND_RE})
- new net ND_WE_N: R131.2, R132.2, U2.G4 (~{ND_WE})
- new net P0_LED_0: R149.2, R150.2, U2.AA17 (ESW_P0_LED_0)
- new net P0_LED_1: R155.2, R156.2, U2.W16 (ESW_P0_LED_1)
- new net P1_LED_0: R151.2, R152.2, U2.Y16 (ESW_P1_LED_0)
- new net P2A_N: J3.2, TR3.14 (MX4+)
- new net P2A_P: J3.1, TR3.13 (MX4-)
- new net P2B_N: J3.6, TR3.18 (CT)
- new net P2B_P: J3.3, TR3.17 (MX3+)
- new net P2C_N: J3.5, TR3.20 (MX2+)
- new net P2C_P: J3.4, TR3.19 (MX2-)
- new net P2D_N: J3.8, TR3.24 (CT)
- new net P2D_P: J3.7, TR3.23 (MX1+)
- new net P3A_N: J2.2, TR2.14 (MX4+)
- new net P3A_P: J2.1, TR2.13 (MX4-)
- new net P3B_N: J2.6, TR2.18 (CT)
- new net P3B_P: J2.3, TR2.17 (MX3+)
- new net P3C_N: J2.5, TR2.20 (MX2+)
- new net P3C_P: J2.4, TR2.19 (MX2-)
- new net P3D_N: J2.8, TR2.24 (CT)
- new net P3D_P: J2.7, TR2.23 (MX1+)
- new net P4A_N: J1.2, TR1.14 (MX4+)
- new net P4A_P: J1.1, TR1.13 (MX4-)
- new net P4B_N: J1.6, TR1.18 (CT)
- new net P4B_P: J1.3, TR1.17 (MX3+)
- new net P4C_N: J1.5, TR1.20 (MX2+)
- new net P4C_P: J1.4, TR1.19 (MX2-)
- new net P4D_N: J1.8, TR1.24 (CT)
- new net P4D_P: J1.7, TR1.23 (MX1+)
- new net PCIE_CK0_N: J5.11 (REFCLK-), R105.1, R110.1
- new net PCIE_CK0_P: J5.13 (REFCLK+), R104.1, R109.1
- new net PCIE_CK1_N: J10.53 (REFCLKn), R107.1, R112.1
- new net PCIE_CK1_P: J10.55 (REFCLKp), R106.1, R111.1
- new net PCIE_CK2_N: R70.1, R71.1, TP29.1
- new net PCIE_CK2_P: R68.1, R69.1, TP28.1
- new net PCIE_RX0_N: C171.2, J5.23 (PERn0)
- new net PCIE_RX0_P: C170.2, J5.25 (PERp0)
- new net PCIE_RX1_N: C173.2, J10.41 (PERn0/SATA-B+)
- new net PCIE_RX1_P: C172.2, J10.43 (PERp0/SATA-B-)
- new net PCIE_RX2_N: C114.2, J10.29 (PERn1)
- new net PCIE_RX2_P: C113.2, J10.31 (PERp1)
- new net PCIE_TX0_N: C165.2, J5.31 (PETn0)
- new net PCIE_TX0_P: C164.2, J5.33 (PETp0)
- new net PCIE_TX1_N: C167.2, J10.47 (PETn0/SATA-A-)
- new net PCIE_TX1_P: C166.2, J10.49 (PETp0/SATA-A+)
- new net PCIE_TX2_N: C112.2, J10.35 (PETn1)
- new net PCIE_TX2_P: C111.2, J10.37 (PETp1)
- new net PERST_N: R137.2, R138.2, R162.2, R3.1, R3.1, U2.G14 (PERST_N)
- new net POWER_LED: U2.W18 (GE2_TXD0)
- new net RA0: U2.E14 (RA0), U9.N3 (A0)
- new net RA1: U2.B18 (RA1), U9.P7 (A1)
- new net RA10: U2.E13 (RA10), U9.L7 (A10/AP)
- new net RA11: U2.C18 (RA11), U9.R7 (A11)
- new net RA12: U2.D15 (RA12), U9.N7 (A12/~{BC})
- new net RA13: U2.B13 (RA13), U9.T3 (A13)
- new net RA14: U2.C17 (RA14), U9.T7 (A14)
- new net RA2: U2.D14 (RA2), U9.P3 (A2)
- new net RA3: U2.A16 (RA3), U9.N2 (A3)
- new net RA4: U2.E15 (RA4), U9.P8 (A4)
- new net RA5: U2.B16 (RA5), U9.P2 (A5)
- new net RA6: U2.D17 (RA6), U9.R8 (A6)
- new net RA7: U2.E11 (RA7), U9.R2 (A7)
- new net RA8: U2.D16 (RA8), U9.T8 (A8)
- new net RA9: U2.D13 (RA9), U9.R3 (A9)
- new net RBA0: U2.C16 (RBA0), U9.M2 (BA0)
- new net RBA1: U2.B17 (RBA1), U9.N8 (BA1)
- new net RBA2: U2.A13 (RBA2), U9.M3 (BA2)
- new net RCKE: U2.A17 (RCKE), U9.K9 (CKE)
- new net RCLK: R34.2, U2.C9 (RCLK), U9.J7 (CK)
- new net RDQ0: U2.C11 (RDQ0), U9.E3 (DQ0)
- new net RDQ1: U2.B3 (RDQ1), U9.F7 (DQ1)
- new net RDQ10: U2.B4 (RDQ10), U9.C8 (DQ10)
- new net RDQ11: U2.B10 (RDQ11), U9.C2 (DQ11)
- new net RDQ12: U2.A5 (RDQ12), U9.A7 (DQ12)
- new net RDQ13: U2.B9 (RDQ13), U9.A2 (DQ13)
- new net RDQ14: U2.C5 (RDQ14), U9.B8 (DQ14)
- new net RDQ15: U2.C8 (RDQ15), U9.A3 (DQ15)
- new net RDQ2: U2.A11 (RDQ2), U9.F2 (DQ2)
- new net RDQ3: U2.A2 (RDQ3), U9.F8 (DQ3)
- new net RDQ4: U2.B12 (RDQ4), U9.H3 (DQ4)
- new net RDQ5: U2.B2 (RDQ5), U9.H8 (DQ5)
- new net RDQ6: U2.C12 (RDQ6), U9.G2 (DQ6)
- new net RDQ7: U2.C2 (RDQ7), U9.H7 (DQ7)
- new net RDQ8: U2.A3 (RDQ8), U9.D7 (DQ8)
- new net RDQ9: U2.C10 (RDQ9), U9.C3 (DQ9)
- new net RDQM0: U2.B5 (RDQM0), U9.E7 (LDM)
- new net RDQM1: U2.B8 (RDQM1), U9.D3 (UDM)
- new net RDQS0: U2.A7 (RDQS0), U9.F3 (LDQS)
- new net RDQS1: U2.C7 (RDQS1), U9.C7 (UDQS)
- new net RODT: U2.B14 (RODT), U9.K1 (ODT)
- new net RTS2: J6.5 (Pin_5), R96.1
- new net RTS2_N: R141.2, R142.2, R96.2, U2.J3 (RTS2_N)
- new net RTS3_N: R143.2, R144.2, TP22.1, U2.J4 (RTS3_N)
- new net SCL: R123.1, R167.1, R98.2, TP33.1, U15.11 (L1), U16.18 (D0)
- new net SDA: R122.1, R166.1, R99.1, TP32.1, U15.12 (L2), U16.19 (D1), U16.20 (D2)
- new net SSUSB_RXN: J8.A10 (RX2-), J8.B10 (RX1-), U13.2 (D-), U2.N3 (SSUSB_RXN)
- new net SSUSB_RXP: J8.A11 (RX2+), J8.B11 (RX1+), U13.1 (D+), U2.N2 (SSUSB_RXP)
- new net SSUSB_TXN: C159.1, U14.2 (D-), U2.M1 (SSUSB_TXN)
- new net SSUSB_TXP: C160.2, U14.1 (D+), U2.M2 (SSUSB_TXP)
- new net TXD1: R145.2, R146.2, R91.2, U2.R14 (TXD1)
- new net TXD2: R139.2, R140.2, R93.2, U2.H2 (TXD2)
- new net UART0_RXD: J6.2 (Pin_2), R92.1
- new net UART0_TXD: J6.1 (Pin_1), R91.1
- new net UART1_RXD: J6.4 (Pin_4), R94.1
- new net UART1_TXD: J6.3 (Pin_3), R93.1
- new net USB1_DM: J5.38 (USB_D+), U2.K1 (USB_DM_P1)
- new net USB1_DP: J5.36 (USB_D-), U2.K2 (USB_DP_P1)
- new net USB_DM: J8.A7 (D-), J8.B7 (D-), U12.2 (D-), U2.M4 (USB_DM_P0)
- new net USB_DP: J8.A6 (D+), J8.B6 (D+), U12.1 (D+), U2.M5 (USB_DP_P0)
- new net VBUS: C120.1, J9.A4 (VBUS), J9.A9 (VBUS), J9.B4 (VBUS), J9.B9 (VBUS), JP1.2 (B), Q1.1 (D1), Q1.2 (D1), Q1.5 (D1), Q1.6 (D1), Q1.8 (D1), U15.32 (VBUS)
- new net VBUSG: Q1.3 (G1), R115.2, U15.33 (VBUSG)
- new net VD: C1.1, C15.1, C17.1, C18.1, C19.1, C23.1, C4.1, C5.1, Q2.1 (D1), Q2.2 (D1), Q2.5 (D1), Q2.6 (D1)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
- new net VMID: C184.1, C186.1, JP1.1 (A), Q1.4 (S1), Q1.7 (S1), R115.1, R117.1, U15.25 (VSN)
- new net VREG: C52.2, R121.2, R122.2, R123.2, U15.27 (VREG)
- new net VSYS: C183.1, R117.2, U15.22 (VSYS), U15.23 (VSYS), U15.24 (VSP), U15.8 (VSYS), U15.9 (VSYS)
- new net WPS: D3.2 (A), R125.2, U2.G15 (WDT_RST_N)
- new net Y0-: U2.Y17 (GE2_TXD3)
- new net Y1-: U2.Y18 (GE2_TXD2)
- new net Y2-: J1.11, U2.W17 (GE2_TXD1)
- new net Y3-: J2.11
- new net Y4-: J3.11
- new net ~{RCAS}: U2.C15 (~{RCAS}), U9.K3 (~{CAS})
- new net ~{RCLK}: R34.1, U2.D9 (~{RCLK}), U9.K7 (~{CK})
- new net ~{RCS}: U2.B15 (~{RCS}), U9.L2 (~{CS})
- new net ~{RDQS0}: U2.B7 (~{RDQS0}), U9.G3 (~{LDQS})
- new net ~{RDQS1}: U2.B6 (~{RDQS1}), U9.B7 (~{UDQS})
- new net ~{RRAS}: U2.C14 (~{RRAS}), U9.J3 (~{RAS})
- new net ~{RWE}: U2.A15 (~{RWE}), U9.L3 (~{WE})
- no-connect marks 0 -> 46
Other:
- removed sheet Charger
- removed sheet Ethernet
- removed sheet Interface
- removed sheet Memory
- removed sheet Other
- removed sheet Power
- note added: "!!!"
- note added: "!!!!!!!!!!!!"
- note added: "SPI_CLK"
- note added: "SPI_CS0_N"
- note added: "SPI_CS1_N"

Commit message: update 100923
Parts:
- removed C133, C137, C138: 4.7u, Capacitor_SMD:C_0603_1608Metric, symbol Device:C_Small
- removed C197: 100n, Capacitor_SMD:C_0402_1005Metric, symbol Device:C_Small
- removed R162, R172: ~, Resistor_SMD:R_0402_1005Metric, symbol Device:R_Small
- removed R163, R166, R167: 4.7k, Resistor_SMD:R_0402_1005Metric, symbol Device:R_Small
- removed R164: 910k, Resistor_SMD:R_0402_1005Metric, symbol Device:R_Small
- removed R165, R168, R169, R170, R171, R98, R99: 0R, Resistor_SMD:R_0402_1005Metric, symbol Device:R_Small
- removed SW4: TS-1187A-B-A-B, Button_Switch_SMD:SW_SPST_TL3342, symbol Switch:SW_Push
- removed TP20, TP21, TP22, TP32, TP33, TP34: TP, MAS_Package_std:TestPoint_Pad_D1mm, symbol Connector:TestPoint
- removed U1: SN74LVC1G175, Package_TO_SOT_SMD:SOT-23-6, symbol MAS_IC_Logic:SN74LVC1G175
- removed U16: N096-2864KSWEG01-H30, MAS_Package_nostd:SSD1306-oled-0.96, symbol MAS_Module:SSD1306-OLED-0.96
- added R76, R77, R78, R79: 22R, Resistor_SMD:R_0402_1005Metric, symbol Device:R_Small
- added R80, R81, R82, R83: 0R, Resistor_SMD:R_0402_1005Metric, symbol Device:R_Small
- added R84, R85, R86: 4.7k, Resistor_SMD:R_0402_1005Metric, symbol Device:R_Small
- added U1: SSD1306-OLED-0.91, MAS_Package_nostd:SSD1306-oled-0.91, symbol MAS_Module:SSD1306-OLED-0.91
- C129: value 4.7u -> 1u; Voltage 16v -> 50v; lcsc C19666 -> C15849
- C130: value 4.7u -> 100n; footprint Capacitor_SMD:C_0603_1608Metric -> Capacitor_SMD:C_0402_1005Metric; Coefficient X5R -> X7R; Voltage 16v -> 50v; lcsc C19666 -> C307331
- C9: value 100n -> 1u; footprint Capacitor_SMD:C_0402_1005Metric -> Capacitor_SMD:C_0603_1608Metric; Coefficient X7R -> X5R; lcsc C307331 -> C15849
- R12: value 1k -> ~; Coefficient 1% -> (none); lcsc C11702 -> (none)
- R87: now not fitted; now left out of the parts list
- renumbered C52 to C126, D1 to D2, D3 to D4, R3 to R17, R3 to R72, R3 to R73, R116 to R75
Connections:
- net +3V3: now also R84.2, R85.2
- net +BATT: no longer R12.2
- net -BATT: now also C130.2, C132.2, U1.7 (VSS); no longer C132.1, C9.2
- net PERST_N: now also R12.2
- net POWER_LED: now also R5.1
- net RTS3_N: now also R79.2
- net at U2.H3 (RXD3): now also R77.2
- net at D4.1 (K), SW2.2: now also Q2.3 (G1), Q3.3 (D), R4.2, TP19.1; no longer C9.1, R12.1
- net at U2.H1 (TXD3): now also R76.2; no longer TP19.1
- net at U2.H5 (CTS3_N): now also R78.2
- net I2C_SCL: now reaches U2.P13 (I2C_SCLK)
- net I2C_SCL: now also R80.2, R82.1, R85.1, U1.10 (SCL)
- net at C129.2: now also U1.3 (C1P)
- net at C129.1: now also U1.4 (C1N)
- net at C130.1: now also R12.1, R86.1, U1.9 (RES#)
- net I2C_SDA: now reaches U2.P14 (I2C_SD)
- net I2C_SDA: now also R81.1, R83.2, R84.1, U1.11 (SDA)
- net UART3_RTS: now reaches J10.30 (NC)
- net UART3_RTS: now also R79.1
- net UART3_CTS: now reaches J10.32 (NC)
- net UART3_CTS: now also R78.1
- net UART3_RXD: now reaches J10.34 (NC)
- net UART3_RXD: now also R77.1
- net UART3_TXD: now reaches J10.36 (NC)
- net UART3_TXD: now also R76.1
- net at J10.56 (NC): now also R83.1
- net at J10.58 (NC): now also R82.2
- net 3V3O: no longer names the net of C131.1, C196.1, R161.1
- net 3V3O: now also R86.2, U1.14 (VCC), U1.5 (VBAT), U1.8 (VDD); no longer C132.2
- net CTS2 renamed UART1_CTS
- net INT renamed PB_INT
- net RTS2 renamed UART1_RTS
- net SCL: no longer names the net of R123.1, U15.11 (L1)
- net SCL: now also R80.1
- net SDA: no longer names the net of R122.1, U15.12 (L2)
- net SDA: now also R81.2
- new net: C132.1, U1.13 (VCOMH)
- new net: C9.1, U1.1 (C2P)
- new net: C9.2, U1.2 (C2N)
- no-connect marks 46 -> 38
Other:
- note added: "I2C/UART no STD!"
- moved on the sheet: C122, C131, C196, C81, C82, D4, R125, R161, R90, R91, R92, SW2

Commit message: update sch
Parts:
- removed J6, J7: IDC-08M, Connector_PinHeader_1.27mm:PinHeader_2x04_P1.27mm_Vertical, symbol Connector_Generic:Conn_02x04_Counter_Clockwise
- removed Q2: SSM6J501NU, MAS_Package_std:U-MOSVI, symbol MAS_Transistors:SSM6J501NU
- removed RN1: 4D03WGJ0102T5E, Resistor_SMD:R_Array_Convex_4x0603, symbol Device:R_Pack04
- added C133: 100n, Capacitor_SMD:C_0402_1005Metric, symbol Device:C_Small
- added C137, C138, C142: 33p, Capacitor_SMD:C_0402_1005Metric, symbol Device:C_Small
- added D5: MBR0540, Diode_SMD:D_SOD-123, symbol Diode:MBR0540
- added J7: ~, Connector_PinHeader_1.27mm:PinHeader_2x05_P1.27mm_Vertical, symbol Connector_Generic:Conn_02x05_Counter_Clockwise
- added J?: 1042240820, MAS_Package_std:1042240820, symbol Connector:SIM_Card_Shielded
- added R126, R127, R162, R163: 4.7k, Resistor_SMD:R_0402_1005Metric, symbol Device:R_Small
- added R88, R89: 0R, Resistor_SMD:R_0402_1005Metric, symbol Device:R_Small
- added R98: 330k, Resistor_SMD:R_0402_1005Metric, symbol Device:R_Small
- added R99: 10k, Resistor_SMD:R_0402_1005Metric, symbol Device:R_Small
- added TP20, TP21, TP22, TP32, TP33, TP34: TP, MAS_Package_std:TestPoint_Pad_D1mm, symbol Connector:TestPoint
- C2: value 100n -> 10u; footprint Capacitor_SMD:C_0402_1005Metric -> Capacitor_SMD:C_0603_1608Metric; Coefficient X7R -> X5R; Voltage 50v -> 10v; lcsc C307331 -> C19702
- R1: value 1k -> 22R; lcsc C11702 -> C25092
- R4: value 10k -> 1k; lcsc C25744 -> C11702
- R5: value 470R -> 22R; Coefficient 5% -> 1%; lcsc C25117 -> C25092
- R7: value 1k -> 470R; Coefficient 1% -> 5%; lcsc C11702 -> C25117
Connections:
- net EN_DC is gone; now on net Y3-: U2.V16 (GE2_TXEN)
- net VD is gone; now on net +BATT: C1.1, C15.1, C17.1, C18.1, C19.1, C23.1, C4.1, C5.1, U3.10 (VIN), U3.11 (VIN), U4.10 (VIN), U4.11 (VIN)
- net Y0- is gone; now on net G2-: U2.Y17 (GE2_TXD3)
- net Y1- is gone; now on net G3-: U2.Y18 (GE2_TXD2)
- net +3V3: now also J7.3 (Pin_3), R126.1, R127.1, R162.1, R163.1
- net +BATT: now also SW2.2; no longer C2.1, R4.1
- net -BATT: now also R4.2, C133.2, C137.2, C138.2, C142.2, J7.4 (Pin_4), J?.5 (GND), J?.SH, R98.1, R99.2; no longer SW2.1
- net D2DB_PORST_N: now also U3.14 (PG), J7.2 (Pin_2)
- net G4-: now also U2.W17 (GE2_TXD1)
- net I2C_SCL: now also R89.1
- net I2C_SDA: now also R88.2
- net PB_INT: now also U2.T18 (GE2_RXD1); no longer U2.V18 (GE2_TXCLK)
- net UART0_RXD: now also J7.6 (Pin_6)
- net UART0_TXD: now also J7.5 (Pin_5)
- net UART1_CTS: now also J5.3 (COEX1)
- net UART1_RTS: now also J5.5 (COEX2)
- net UART1_RXD: now also J5.45 (Reserved)
- net UART1_TXD: now also J5.51 (Reserved)
- net USB1_DM: now also J5.36 (USB_D-); no longer J5.38 (USB_D+)
- net USB1_DP: now also J5.38 (USB_D+); no longer J5.36 (USB_D-)
- net WPS: now also Q3.3 (D); no longer D4.2 (A)
- net Y2-: now also U2.W18 (GE2_TXD0); no longer U2.W17 (GE2_TXD1)
- net Y4-: now also U2.V18 (GE2_TXCLK)
- net at C20.1, R6.2, U3.1 (VINA): no longer R1.2
- net at U2.R17 (GE2_RXCLK): now also TP34.1
- net at U2.T16 (GE2_RXDV): now also TP33.1
- net at U2.T17 (GE2_RXD0): now also TP32.1
- net at U2.U15 (MDIO): now also TP22.1
- net PWR5V_ON: now reaches U2.U16 (GE2_RXD2)
- net PWR5V_ON: now also R1.1
- net PWR_ON: now reaches U2.U17 (GE2_RXD3)
- net PWR_ON: now also D5.2 (A)
- net at R97.1: now also J7.9 (Pin_9), R162.2
- net at C21.1, R16.2, U4.1 (VINA): no longer R7.2
- net at TP18.1: now also J5.17 (UIM_C8); no longer J5.51 (Reserved)
- net at U3.12 (EN): now also R1.2, R4.1; no longer R1.1
- net at R7.1: now also D4.2 (A), Q3.1 (G), R99.1; no longer U4.12 (EN)
- net at R5.2: now also U4.12 (EN); no longer Q3.1 (G)
- net at TP17.1: now also J5.19 (UIM_C4); no longer J5.45 (Reserved)
- net at U2.F16 (JTCLK): now also J7.1 (Pin_1), R126.2
- net at R90.2, U2.F17 (JTRST_N): now also J7.7 (Pin_7)
- net at U2.G16 (JTDI): now also J7.8 (Pin_8), R163.2
- net at U2.G18 (JTMS): now also J7.10 (Pin_10), R127.2
- net UIM_DATA: now reaches J5.10 (UIM_DATA)
- net UIM_DATA: now also C142.1, J?.7 (I/O)
- net UIM_CLK: now reaches J5.12 (UIM_CLK)
- net UIM_CLK: now also C138.1, J?.3 (CLK)
- net UIM_RST: now reaches J5.14 (~{UIM_RESET})
- net UIM_RST: now also C137.1, J?.2 (RST)
- net UIM_VPP: now reaches J5.16 (UIM_VPP)
- net UIM_VPP: now also J?.6 (VPP)
- net at J5.30 (SMB_CLK): now also R89.2
- net at J5.32 (SMB_DATA): now also R88.1
- net at J5.42 (~{LED_WWAN}): now also TP21.1
- net at J5.46 (~{LED_WPAN}): now also TP20.1
- net UIM_PWR: now reaches J5.8 (UIM_PWR)
- net UIM_PWR: now also C133.1, J?.1 (VCC)
- net POWER_LED renamed PWR3V_ON
- net PWR3V_ON: now also C2.1, D4.1 (K), TP19.1, D5.1 (K), R98.2; no longer U2.W18 (GE2_TXD0)
- new net: R7.2, SW2.1
- no-connect marks 38 -> 17
Other:
- note added: "UART no STD!"
- note removed: "!!!!!!!!!!!!"
- moved on the sheet: C121, C20, C21, C76, D2, D4, Q3, R125, R3, R75, R90, SW2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

Commit message: update pcb
Parts:
- removed R97: 22R, Resistor_SMD:R_0402_1005Metric, symbol Device:R_Small
Connections:
- net at J7.9 (Pin_9), R162.2: now also U2.G17 (JTDO)
Other:
- moved on the sheet: C1, C10, C100, C101, C102, C103, C104, C105, C106, C107, C108, C109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

Commit message: update pcb
Parts:
- J8: footprint Connector_USB:USB_C_Receptacle_HRO_TYPE-C-31-M-12 -> MAS_Package_std:HRS_CX90B1-24P; description (none) -> C5178546; lcsc (none) -> C2681555
Connections:
- net +5V: now also C33.1
- net -BATT: now also J10.S1 (MP), J10.S2 (MP)
- net SSUSB_TXN: no longer U14.2 (D-)
- net SSUSB_TXP: no longer U14.1 (D+)
- net at C28.1, C6.1, JP2.2 (B)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: no longer C33.1
- net at C160.1, J8.A2 (TX1+), J8.B2 (TX2+): now also U14.1 (D+)
- net at C159.2, J8.A3 (TX1-), J8.B3 (TX2-): now also U14.2 (D-)
Other:
- moved on the sheet: C159, C160, C33, JP2

Commit message: updated rules for differential pairs
Connections:
- net SSUSB_RXN: now also U13.1 (D+); no longer U13.2 (D-)
- net SSUSB_RXP: now also U13.2 (D-); no longer U13.1 (D+)
- net USB1_DM: no longer U2.K1 (USB_DM_P1)
- net _PCIE_TX0_P: now reaches C164.1, U2.L18 (PCIE_TXP1)
- net _SSUSB_TXP: now reaches C160.1, J8.A2 (TX1+), J8.B2 (TX2+), U14.1 (D+)
- net _SSUSB_TXN: now reaches C159.2, J8.A3 (TX1-), J8.B3 (TX2-), U14.2 (D-)
- net _PCIE_CK2_P: now reaches R69.2, U2.M13 (PCIE_CKP2)
- net _PCIE_TX2_N: now reaches C112.1, U2.N17 (PCIE_TXN2)
- net _PCIE_CK0_N: now reaches R105.2, U2.K14 (PCIE_CKN1)
- net _PCIE_CK1_N: now reaches R107.2, U2.H13 (PCIE_CKN0)
- net _PCIE_TX2_P: now reaches C111.1, U2.N16 (PCIE_TXP2)
- net _PCIE_TX1_N: now reaches C167.1, U2.H17 (PCIE_TXN0)
- net _PCIE_CK0_P: now reaches R104.2, U2.K13 (PCIE_CKP1)
- net _PCIE_CK1_P: now reaches R106.2, U2.H14 (PCIE_CKP0)
- net _PCIE_TX1_P: now reaches C166.1, U2.H16 (PCIE_TXP0)
- net _PCIE_RX1_N: now reaches C173.1, U2.J16 (PCIE_RXN0)
- net _PCIE_RX1_P: now reaches C172.1, U2.J17 (PCIE_RXP0)
- net _PCIE_RX0_N: now reaches C171.1, U2.K16 (PCIE_RXN1)
- net _PCIE_RX0_P: now reaches C170.1, U2.K17 (PCIE_RXP1)
- net _PCIE_TX0_N: now reaches C165.1, U2.L17 (PCIE_TXN1)
- net _PCIE_CK2_N: now reaches R70.2, U2.M14 (PCIE_CKN2)
- net _PCIE_RX2_P: now reaches C113.1, U2.M17 (PCIE_RXP2)
- net _PCIE_RX2_N: now reaches C114.1, U2.M18 (PCIE_RXN2)
- net ESW_TXVN_A_P2 renamed ESW_A_P2_TXVN
- net ESW_TXVN_A_P3 renamed ESW_A_P3_TXVN
- net ESW_TXVN_A_P4 renamed ESW_A_P4_TXVN
- net ESW_TXVN_B_P2 renamed ESW_B_P2_TXVN
- net ESW_TXVN_B_P3 renamed ESW_B_P3_TXVN
- net ESW_TXVN_B_P4 renamed ESW_B_P4_TXVN
- net ESW_TXVN_C_P2 renamed ESW_C_P2_TXVN
- net ESW_TXVN_C_P3 renamed ESW_C_P3_TXVN
- net ESW_TXVN_C_P4 renamed ESW_C_P4_TXVN
- net ESW_TXVN_D_P2 renamed ESW_D_P2_TXVN
- net ESW_TXVN_D_P3 renamed ESW_D_P3_TXVN
- net ESW_TXVN_D_P4 renamed ESW_D_P4_TXVN
- net ESW_TXVP_A_P2 renamed ESW_A_P2_TXVP
- net ESW_TXVP_A_P3 renamed ESW_A_P3_TXVP
- net ESW_TXVP_A_P4 renamed ESW_A_P4_TXVP
- net ESW_TXVP_B_P2 renamed ESW_B_P2_TXVP
- net ESW_TXVP_B_P3 renamed ESW_B_P3_TXVP
- net ESW_TXVP_B_P4 renamed ESW_B_P4_TXVP
- net ESW_TXVP_C_P2 renamed ESW_C_P2_TXVP
- net ESW_TXVP_C_P3 renamed ESW_C_P3_TXVP
- net ESW_TXVP_C_P4 renamed ESW_C_P4_TXVP
- net ESW_TXVP_D_P2 renamed ESW_D_P2_TXVP
- net ESW_TXVP_D_P3 renamed ESW_D_P3_TXVP
- net ESW_TXVP_D_P4 renamed ESW_D_P4_TXVP
- net RCLK renamed RCLK_P
- net RDQS0 renamed RDQS0_P
- net RDQS1 renamed RDQS1_P
- net USB_DM renamed USB_DN
- net ~{RCLK} renamed RCLK_N
- net ~{RDQS0} renamed RDQS0_N
- net ~{RDQS1} renamed RDQS1_N
- new net USB1_DN: U2.K1 (USB_DM_P1)
Other:
- moved on the sheet: C111, C112, C113, C114, C164, C165, C166, C167, C170, C171, C172, C173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

Commit message: calc Impedance and mark wire
Connections:
- net USB1_DM is gone; now on net USB1_DN: J5.36 (USB_D-)
- net JTDO: now reaches J7.9 (Pin_9), R162.2, U2.G17 (JTDO)
- net JTDI: now reaches J7.8 (Pin_8), R163.2, U2.G16 (JTDI)
- net _UART3_TXD: now reaches R76.2, U2.H1 (TXD3)
- net JTCLK: now reaches J7.1 (Pin_1), R126.2, U2.F16 (JTCLK)
- net JTMS: now reaches J7.10 (Pin_10), R127.2, U2.G18 (JTMS)
- net JTRST_N: now reaches J7.7 (Pin_7), R90.2, U2.F17 (JTRST_N)
- net _UART3_RXD: now reaches R77.2, U2.H3 (RXD3)
- net _UART0_RXD: now reaches R92.2, U2.R13 (RXD1)
- net _UART1_RXD: now reaches R94.2, U2.H4 (RXD2)
- net _UART3_CTS: now reaches R78.2, U2.H5 (CTS3_N)
- net _UART1_CTS: now reaches R95.2, U2.J5 (CTS2_N)
- net DDR3RSTB renamed DDR_STB
- net ND_CS_N renamed SPI_CS_N
- net ND_D4 renamed SPI_D4
- net ND_D5 renamed SPI_D5
- net ND_D6 renamed SPI_D6
- net ND_D7 renamed SPI_D7
- net ND_RE_N renamed SPI_RE_N
- net ND_WE_N renamed SPI_WE_N
- net P2A_N renamed ESW_P2A_N
- net P2A_P renamed ESW_P2A_P
- net P2B_N renamed ESW_P2B_N
- net P2B_P renamed ESW_P2B_P
- net P2C_N renamed ESW_P2C_N
- net P2C_P renamed ESW_P2C_P
- net P2D_N renamed ESW_P2D_N
- net P2D_P renamed ESW_P2D_P
- net P3A_N renamed ESW_P3A_N
- net P3A_P renamed ESW_P3A_P
- net P3B_N renamed ESW_P3B_N
- net P3B_P renamed ESW_P3B_P
- net P3C_N renamed ESW_P3C_N
- net P3C_P renamed ESW_P3C_P
- net P3D_N renamed ESW_P3D_N
- net P3D_P renamed ESW_P3D_P
- net P4A_N renamed ESW_P4A_N
- net P4A_P renamed ESW_P4A_P
- net P4B_N renamed ESW_P4B_N
- net P4B_P renamed ESW_P4B_P
- net P4C_N renamed ESW_P4C_N
- net P4C_P renamed ESW_P4C_P
- net P4D_N renamed ESW_P4D_N
- net P4D_P renamed ESW_P4D_P
- net RA0 renamed DDR_A0
- net RA1 renamed DDR_A1
- net RA10 renamed DDR_A10
- net RA11 renamed DDR_A11
- net RA12 renamed DDR_A12
- net RA13 renamed DDR_A13
- net RA14 renamed DDR_A14
- net RA2 renamed DDR_A2
- net RA3 renamed DDR_A3
- net RA4 renamed DDR_A4
- net RA5 renamed DDR_A5
- net RA6 renamed DDR_A6
- net RA7 renamed DDR_A7
- net RA8 renamed DDR_A8
- net RA9 renamed DDR_A9
- net RBA0 renamed DDR_BA0
- net RBA1 renamed DDR_BA1
- net RBA2 renamed DDR_BA2
- net RCKE renamed DDR_CKE
- net RCLK_N renamed DDR_CLK_N
- net RCLK_P renamed DDR_CLK_P
- net RDQ0 renamed DDR_Q0
- net RDQ1 renamed DDR_Q1
- net RDQ10 renamed DDR_Q10
- net RDQ11 renamed DDR_Q11
- net RDQ12 renamed DDR_Q12
- net RDQ13 renamed DDR_Q13
- net RDQ14 renamed DDR_Q14
- net RDQ15 renamed DDR_Q15
- net RDQ2 renamed DDR_Q2
- net RDQ3 renamed DDR_Q3
- net RDQ4 renamed DDR_Q4
- net RDQ5 renamed DDR_Q5
- net RDQ6 renamed DDR_Q6
- net RDQ7 renamed DDR_Q7
- net RDQ8 renamed DDR_Q8
- net RDQ9 renamed DDR_Q9
- net RDQM0 renamed DDR_QM0
- net RDQM1 renamed DDR_QM1
- net RDQS0_N renamed DDR_QS0_N
- net RDQS0_P renamed DDR_QS0_P
- net RDQS1_N renamed DDR_QS1_N
- net RDQS1_P renamed DDR_QS1_P
- net RODT renamed DDR_ODT
- net RTS2_N renamed _UART1_RTS
- net RTS3_N renamed _UART3_RTS
- net SSUSB_RXN renamed USB_RXN
- net SSUSB_RXP renamed USB_RXP
- net SSUSB_TXN renamed USB_TXN
- net SSUSB_TXP renamed USB_TXP
- net TXD1 renamed _UART0_TXD
- net TXD2 renamed _UART1_TXD
- net _SSUSB_TXN renamed _USB_TXN
- net _SSUSB_TXP renamed _USB_TXP
- net ~{RCAS} renamed DDR_~{CAS}
- net ~{RCS} renamed DDR_~{CS}
- net ~{RRAS} renamed DDR_~{RAS}
- net ~{RWE} renamed DDR_~{WE}
Other:
- company: (none) -> FOSS
- title: (none) -> Open pocket router
- moved on the sheet: R93, R94, R95, R96
